File: maglock.kicad_pcb (KiCad board)
At the start: 2 copper layers, 98 x 98 mm, 157 parts, among them J1 USB_UART, J2 USB, J3 Lock, J4 Door Open, J5 Door Close, J6 Power IN, J8 5V_2, K1 FINDER-36.11, K2 FINDER-36.11, K3 FINDER-36.11, Q1 AO3400A, Q2 AO3400A, Q3 AO3400A, Q4 AO3400A, Q5 HYG210P06LQ1D, SW1 2pin, SW2 2pin, SW3 2pin, SW4 2pin, U1 USBLC6-2SC6, U2 3V3 LDO, U3 CH340C, U4 DS18B20Z, U5 USBLC6-2SC6, U6 USBLC6-2SC6, U7 XL4001, U8 XL4001

Commit message: most stuff squeezed on board
Parts:
- removed the C12 at (35.0, 163.0)
- removed the C13 at (65.6, 89.2)
- removed the C14 at (70.3, 161.9)
- removed the D13 at (163.9, 64.3)
- removed the D14 at (164.4, 80.0)
- removed the D15 at (164.4, 96.0)
- removed the F6 at (64.2, 69.7)
- removed the J6 at (64.6, 27.0)
- removed OP1, OP2, OP3: EL817S1(C), Package_DIP:SMDIP-4_W9.53mm
- removed the R37 at (167.4, 55.0)
- removed the R38 at (167.4, 71.0)
- removed the R39 at (167.4, 86.9)
- removed the R55 at (85.5, 120.8)
- removed kibuzzard-62CD9C06: G***, kibuzzard-62CD9C06
- removed kibuzzard-62CDFAFC: G***, kibuzzard-62CDFAFC
- added C18: 10u/35v, Capacitor_SMD:C_1206_3216Metric, F.Cu at (139.4, 76.6)
- added C19: 100n, Capacitor_SMD:C_0805_2012Metric, F.Cu at (133.2, 59.0)
- added C20: 100n, Capacitor_SMD:C_0805_2012Metric, F.Cu at (133.3, 74.3)
- added C24: 10u/35v, Capacitor_SMD:C_1206_3216Metric, F.Cu at (143.1, 55.6)
- added C25: 10u/35v, Capacitor_SMD:C_1206_3216Metric, F.Cu at (145.5, 71.0)
- added C26: 10u/35v, Capacitor_SMD:C_1206_3216Metric, F.Cu at (145.5, 55.6)
- added C27: 10u/35v, Capacitor_SMD:C_1206_3216Metric, F.Cu at (147.9, 71.0)
- added C28: 220u/35v, Capacitor_SMD:CP_Elec_10x10, F.Cu at (123.3, 73.2)
- added C29: 10u/35v, Capacitor_SMD:C_1206_3216Metric, F.Cu at (133.8, 104.1)
- added C30: 10u/35v, Capacitor_SMD:C_1206_3216Metric, F.Cu at (116.7, 93.4)
- added C31: 10u/35v, Capacitor_SMD:C_1206_3216Metric, F.Cu at (155.7, 110.1)
- added C32: 10u/35v, Capacitor_SMD:C_1206_3216Metric, F.Cu at (131.4, 104.1)
- added C33: 10u/35v, Capacitor_SMD:C_1206_3216Metric, F.Cu at (119.0, 93.4)
- added C34: 10u/35v, Capacitor_SMD:C_1206_3216Metric, F.Cu at (155.7, 107.7)
- added C35: 100u/10v, Capacitor_SMD:C_1206_3216Metric, F.Cu at (128.6, 92.0)
- added C36: 100u/10v, Capacitor_SMD:C_1206_3216Metric, F.Cu at (119.0, 98.1)
- added C37: 100u/10v, Capacitor_SMD:C_1206_3216Metric, F.Cu at (150.9, 104.1)
- added C40: 100n, Capacitor_SMD:C_0805_2012Metric, F.Cu at (150.3, 108.3)
- added C43: 100u/10v, Capacitor_SMD:C_1206_3216Metric, F.Cu at (150.9, 101.7)
- added C44: 100u/10v, Capacitor_SMD:C_1206_3216Metric, F.Cu at (128.6, 96.8)
- added C45: 100u/10v, Capacitor_SMD:C_1206_3216Metric, F.Cu at (111.3, 117.1)
- added C46: 100u/10v, Capacitor_SMD:C_1206_3216Metric, F.Cu at (150.9, 99.2)
- added C5: 100u/10v, Capacitor_SMD:C_1206_3216Metric, F.Cu at (162.6, 110.8)
- added C6: 100u/10v, Capacitor_SMD:C_1206_3216Metric, F.Cu at (162.6, 113.3)
- added C7: 100u/10v, Capacitor_SMD:C_1206_3216Metric, F.Cu at (139.6, 129.8)
- added C8: 100u/10v, Capacitor_SMD:C_1206_3216Metric, F.Cu at (162.6, 108.4)
- added D19: SS34A, Diode_SMD:D_SMA, F.Cu at (138.5, 65.4)
- added D20: SS34A, Diode_SMD:D_SMA, F.Cu at (138.5, 80.8)
- added D21: SS34A, Diode_SMD:D_SMA, F.Cu at (145.6, 65.4)
- added D22: SS34A, Diode_SMD:D_SMA, F.Cu at (145.6, 80.8)
- added D26: YELLOW, LED_SMD:LED_0805_2012Metric_Pad1.15x1.40mm_HandSolder, F.Cu at (164.4, 56.4)
- added D27: YELLOW, LED_SMD:LED_0805_2012Metric_Pad1.15x1.40mm_HandSolder, F.Cu at (164.4, 71.8)
- added D30: SS34A, Diode_SMD:D_SMA, F.Cu at (152.2, 113.1)
- added D33: SS34A, Diode_SMD:D_SMA, F.Cu at (160.7, 101.5)
- added D36: RED, LED_SMD:LED_0805_2012Metric_Pad1.15x1.40mm_HandSolder, F.Cu at (164.4, 87.1)
- added F4: 2A, Fuse:Fuse_1206_3216Metric_Pad1.42x1.75mm_HandSolder, F.Cu at (109.3, 80.7)
- added F5: 7A, Inductor_SMD:L_1206_3216Metric_Pad1.42x1.75mm_HandSolder, F.Cu at (116.6, 54.1)
- added F7: 1A, Fuse:Fuse_1206_3216Metric_Pad1.42x1.75mm_HandSolder, F.Cu at (109.3, 88.2)
- added F8: 1A, Fuse:Fuse_1206_3216Metric_Pad1.42x1.75mm_HandSolder, F.Cu at (109.3, 83.2)
- added J10: Power IN, TerminalBlock_Phoenix:TerminalBlock_Phoenix_PT-1,5-4-3.5-H_1x04_P3.50mm_Horizontal, F.Cu at (109.3, 62.1)
- added J11: 12V_1, Connector_PinHeader_2.54mm:PinHeader_1x03_P2.54mm_Vertical, F.Cu at (164.4, 59.2)
- added J12: 12V_2, Connector_PinHeader_2.54mm:PinHeader_1x03_P2.54mm_Vertical, F.Cu at (164.4, 74.7)
- added J13: 5V_1, Connector_PinHeader_2.54mm:PinHeader_1x03_P2.54mm_Vertical, F.Cu at (146.2, 90.1)
- added J15: 5V_3, Connector_PinHeader_2.54mm:PinHeader_1x03_P2.54mm_Vertical, F.Cu at (164.4, 90.0)
- added J2: I2C0_128x32, -local:oled_i2c_128x32_ssd1306, F.Cu at (219.0, 102.2)
- added J3: I2C1, Connector_PinSocket_2.54mm:PinSocket_1x04_P2.54mm_Vertical, F.Cu at (132.9, 127.1)
- added J4: SPI1, Connector_PinSocket_2.54mm:PinSocket_1x06_P2.54mm_Vertical, F.Cu at (145.6, 127.1)
- added J5: I2C0_128x64, -local:oled_i2c_128x64_ssd1306, F.Cu at (228.0, 127.5)
- added L1: 47u/2.5A, -local:L_12x12mm_H8mm__D11.0_P5.0_universal, F.Cu at (155.8, 60.3)
- added L2: 47u/2.5A, -local:L_12x12mm_H8mm__D11.0_P5.0_universal, F.Cu at (155.8, 75.7)
- added L5: 47u/2.5A, -local:L_12x12mm_H8mm__D11.0_P5.0_universal, F.Cu at (155.8, 91.0)
- added R45: 1k, Resistor_SMD:R_0805_2012Metric, F.Cu at (133.2, 63.0)
- added R46: 1k, Resistor_SMD:R_0805_2012Metric, F.Cu at (133.2, 61.0)
- added R47: 1k, Resistor_SMD:R_0805_2012Metric, F.Cu at (133.3, 78.3)
- added R48: 1k, Resistor_SMD:R_0805_2012Metric, F.Cu at (133.3, 76.3)
- added R49: 10k, Resistor_SMD:R_0805_2012Metric, F.Cu at (164.4, 54.4)
- added R50: 10k, Resistor_SMD:R_0805_2012Metric, F.Cu at (164.4, 69.8)
- added R56: 1k5, Resistor_SMD:R_0805_2012Metric, F.Cu at (150.3, 110.3)
- added R59: 1k, Resistor_SMD:R_0805_2012Metric, F.Cu at (164.4, 85.1)
- added RV1: 10k, Potentiometer_THT:Potentiometer_Bourns_3296W_Vertical, F.Cu at (134.2, 55.2)
- added RV2: 10k, Potentiometer_THT:Potentiometer_Bourns_3296W_Vertical, F.Cu at (134.3, 70.6)
- added U11: XL4001, Package_SO:Texas_HTSOP-8-1EP_3.9x4.9mm_P1.27mm_EP2.95x4.9mm_Mask2.4x3.1mm_ThermalVias, F.Cu at (156.1, 102.2)
- added U7: XL4001, Package_SO:Texas_HTSOP-8-1EP_3.9x4.9mm_P1.27mm_EP2.95x4.9mm_Mask2.4x3.1mm_ThermalVias, F.Cu at (144.9, 60.8)
- added U8: XL4001, Package_SO:Texas_HTSOP-8-1EP_3.9x4.9mm_P1.27mm_EP2.95x4.9mm_Mask2.4x3.1mm_ThermalVias, F.Cu at (144.9, 76.2)
- added kibuzzard-62CF1330: G***, kibuzzard-62CF1330, F.Cu at (113.7, 70.9)
- added kibuzzard-62D1D969: G***, kibuzzard-62D1D969, F.Cu at (168.8, 91.3)
- added kibuzzard-62D1D979: G***, kibuzzard-62D1D979, F.Cu at (184.2, 115.7)
- added kibuzzard-62D1D983: G***, kibuzzard-62D1D983, F.Cu at (183.8, 141.2)
- added kibuzzard-62D1E5EA: G***, kibuzzard-62D1E5EA, F.Cu at (121.0, 111.1)
- added kibuzzard-62D1E68D: G***, kibuzzard-62D1E68D, F.Cu at (116.3, 71.1)
- added kibuzzard-62D1EAEB: G***, kibuzzard-62D1EAEB, F.Cu at (109.3, 76.0)
- added kibuzzard-62D2019E: G***, kibuzzard-62D2019E, F.Cu at (167.2, 60.8)
- added kibuzzard-62D201BA: G***, kibuzzard-62D201BA, F.Cu at (167.2, 76.4)
- added kibuzzard-62D201CC: G***, kibuzzard-62D201CC, F.Cu at (130.2, 87.4)
- added kibuzzard-62D2A27A: G***, kibuzzard-62D2A27A, F.Cu at (164.1, 99.0)
- C15, C16, C17: value 1u -> 10u/35v; footprint Capacitor_SMD:C_0805_2012Metric -> Capacitor_SMD:C_1206_3216Metric
- C22, C23: value 1000u/10v -> 10u/35v; footprint Capacitor_SMD:CP_Elec_10x10 -> Capacitor_SMD:C_1206_3216Metric
- C4: value 1000u/10v -> 100u/10v; footprint Capacitor_SMD:CP_Elec_10x10 -> Capacitor_SMD:C_1206_3216Metric
- F3: renamed from F4; value PTC 2A -> 2A; footprint -local:Fuse_2920_7451Metric_Pad2.10x5.45mm_HandSolder -> Fuse:Fuse_1206_3216Metric_Pad1.42x1.75mm_HandSolder
- F6: renamed from F5; value PTC 1A -> 1A; footprint -local:Fuse_2920_7451Metric_Pad2.10x5.45mm_HandSolder -> Fuse:Fuse_1206_3216Metric_Pad1.42x1.75mm_HandSolder
- LOGO2: footprint Symbol:OSHW-Logo2_7.3x6mm_SilkScreen -> Symbol:OSHW-Logo2_9.8x8mm_SilkScreen
- R31, R32, R33: value 100 -> 330
- R53: value 1k -> 4k7
- moved C22 174.2 mm to (147.9, 55.6), turned to -90 degrees
- moved D34 148.9 mm to (146.2, 87.2)
- moved D31 142.0 mm to (142.4, 101.5), turned to -90 degrees
- moved F3 131.7 mm to (109.3, 78.2)
- moved BZ1 130.5 mm to (141.3, 159.4), turned to 0 degrees
- moved C16 127.3 mm to (137.0, 76.6), turned to 90 degrees
- moved U9 125.5 mm to (137.8, 102.2), turned to -90 degrees
- moved F6 125.0 mm to (109.3, 85.7)
- moved R54 117.2 mm to (129.9, 99.7), turned to 90 degrees
- moved C17 116.9 mm to (137.0, 61.2), turned to 90 degrees
- moved R51 116.8 mm to (133.9, 99.7), turned to 90 degrees
- moved C38 116.4 mm to (131.9, 99.7), turned to 90 degrees
- moved R53 113.9 mm to (150.3, 106.3), turned to 180 degrees
- moved L3 113.7 mm to (137.6, 91.0), turned to 90 degrees
- moved C23 107.4 mm to (143.1, 71.0), turned to -90 degrees
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- renumbered C6 to C10, C7 to C11, C8 to C12, C9 to C13, C10 to C14, C11 to C21, C18 to C38, C19 to C39, C20 to C41, C21 to C42, C5 to C9, D16 to D13, D17 to D14, D18 to D15, D19 to D16, D20 to D17, D21 to D18, D22 to D23, D23 to D24, D24 to D25, D25 to D28, D26 to D29, D27 to D31, D28 to D32, D29 to D34, D30 to D35, J8 to J14, J2 to J6, J3 to J7, J4 to J8, J5 to J9, L1 to L3, L2 to L4, R40 to R37, R41 to R38, R42 to R39, R43 to R40, R44 to R41, R45 to R42, R46 to R43, R47 to R44, R48 to R51, R49 to R52, R50 to R54, R51 to R55, R52 to R57, R54 to R58, U8 to U10, U7 to U9
Connections:
- A1 pad MP: (no net) -> GND
- A1 pad a10: unconnected-(A1-Pada10) -> /_MAIN_SOC/REL2
- A1 pad a12: /_MAIN_SOC/_BUZZER -> /_MAIN_SOC/REL1
- A1 pad a16: unconnected-(A1-Pada16) -> /_MAIN_SOC/I2C1_SDA
- A1 pad a18: unconnected-(A1-Pada18) -> /_MAIN_SOC/I2C1_SCK
- A1 pad a19: unconnected-(A1-Pada19) -> /_MAIN_SOC/SPI1_MOSI
- A1 pad a21: unconnected-(A1-Pada21) -> /_MAIN_SOC/SPI1_MISO
- A1 pad a23: unconnected-(A1-Pada23) -> /_MAIN_SOC/SPI1_CLK
- A1 pad a24: unconnected-(A1-Pada24) -> /_MAIN_SOC/SPI1_CS
- A1 pad a3: unconnected-(A1-Pada3) -> /_MAIN_SOC/I2C0_SDA
- A1 pad a5: unconnected-(A1-Pada5) -> /_MAIN_SOC/I2C0_SCK
- A1 pad a7: unconnected-(A1-Pada7) -> /_MAIN_SOC/_BUZZER
- C15 pad 1: /_POWER/VIN2 -> /_POWER/VIN4
- C16 pad 1: /_POWER/VOUT1 -> /_POWER/VIN5
- C17 pad 1: /_POWER/VOUT2 -> /_POWER/VIN4
- C22 pad 1: /_POWER/VOUT1 -> /_POWER/VOUT4
- C23 pad 1: /_POWER/VOUT2 -> /_POWER/VOUT5
- C4 pad 1: /_INPUTS/3V3 -> GND
- C4 pad 2: GND -> /_MAIN_SOC/5V
- F3 pad 1: unconnected-(F4-Pad1) -> /_POWER/VIN
- F3 pad 2: unconnected-(F4-Pad2) -> Net-(D19-Pad2)
- F6 pad 1: unconnected-(F5-Pad1) -> /_POWER/VIN
- J7 pad 1: /_POWER/12V@2A_ADJ_1 -> GND
- J7 pad 3: GND -> /_POWER/12V@2A_ADJ_1
- J8 pad 1: /_POWER/12V@2A_ADJ_2 -> GND
- J8 pad 3: GND -> /_POWER/12V@2A_ADJ_2
- J9 pad 1: /_POWER/12V@2A_ADJ_2 -> GND
- J9 pad 3: GND -> /_POWER/12V@2A_ADJ_2
- K1 pad 12: GND -> /_POWER/12V@2A_ADJ_1
- K1 pad 14: /_POWER/12V@2A_ADJ_1 -> GND
- K2 pad 12: GND -> /_POWER/12V@2A_ADJ_2
- K2 pad 14: /_POWER/12V@2A_ADJ_2 -> GND
- K3 pad 12: GND -> /_POWER/12V@2A_ADJ_2
- K3 pad 14: /_POWER/12V@2A_ADJ_2 -> GND
- Q2 pad 1: Net-(OP1-Pad3) -> Net-(Q2-Pad1)
- Q3 pad 1: Net-(OP2-Pad3) -> Net-(Q3-Pad1)
- Q4 pad 1: Net-(OP3-Pad3) -> Net-(Q4-Pad1)
- R31 pad 2: Net-(OP1-Pad1) -> Net-(Q2-Pad1)
- R32 pad 2: Net-(OP2-Pad1) -> Net-(Q3-Pad1)
- R33 pad 2: Net-(OP3-Pad1) -> Net-(Q4-Pad1)
- R34 pad 1: Net-(OP1-Pad3) -> Net-(Q2-Pad1)
- R35 pad 1: Net-(OP2-Pad3) -> Net-(Q3-Pad1)
- R36 pad 1: Net-(OP3-Pad3) -> Net-(Q4-Pad1)
- R53 pad 1: GND -> /_POWER/FB3
- R53 pad 2: Net-(R52-Pad1) -> /_POWER/VOUT3
- R57 pad 1: Net-(R52-Pad1) -> GND
- R58 pad 1: Net-(R54-Pad1) -> GND
Routing:
- net /_POWER/5V@2A_3: track 0.00 -> 59.0 mm
- net /_INPUTS/SW4: track 0.00 -> 44.6 mm
- net GND: track 25.5 -> 63.9 mm, vias 29 -> 135
- net /_POWER/VOUT2: track 0.00 -> 38.2 mm
- net /_POWER/VOUT3: track 0.00 -> 36.6 mm
- net /_POWER/12V@2A_ADJ_2: track 0.00 -> 32.8 mm
- net /_POWER/VOUT4: track 0.00 -> 31.5 mm
- net /_POWER/VOUT5: track 0.00 -> 31.4 mm
- net /_INPUTS/SW3: track 0.00 -> 26.8 mm
- net /_POWER/FB4: track 0.00 -> 25.0 mm
- net /_POWER/FB5: track 0.00 -> 24.8 mm
- net /_POWER/VIN_E: track 0.00 -> 23.9 mm
- net Net-(J9-Pad2): track 0.00 -> 23.6 mm
- net /_POWER/VIN: track 0.00 -> 23.6 mm
- net Net-(J7-Pad2): track 0.00 -> 22.7 mm
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- added copper zone on F.Cu, net /_POWER/SW1
- added copper zone on F.Cu, net /_POWER/SW2
- added copper zone on F.Cu, net /_POWER/SW3
- added copper zone on F.Cu, net /_POWER/SW4
- added copper zone on F.Cu, net /_POWER/SW5
- added copper zone on F.Cu, net /_POWER/VIN
- added copper zone on F.Cu, net /_POWER/VIN1
- added copper zone on F.Cu, net /_POWER/VIN2
- added copper zone on F.Cu, net /_POWER/VIN3
- added copper zone on F.Cu, net /_POWER/VIN4
- added copper zone on F.Cu, net /_POWER/VIN5
- added copper zone on F.Cu, net /_POWER/VOUT1
- added copper zone on F.Cu, net /_POWER/VOUT2
- added copper zone on F.Cu, net /_POWER/VOUT4
- added copper zone on F.Cu, net /_POWER/VOUT5
- added copper zone on F.Cu, net GND

Commit message: general routing finished
Parts:
- removed the C7 at (139.6, 129.8)
- removed kibuzzard-62CF1330: G***, kibuzzard-62CF1330
- removed kibuzzard-62D2A27A: G***, kibuzzard-62D2A27A
- added JP1: IO power selector, Jumper:SolderJumper-3_P1.3mm_Open_RoundedPad1.0x1.5mm, F.Cu at (156.4, 126.1)
- added R13: 100, Resistor_SMD:R_0805_2012Metric, F.Cu at (162.0, 124.7)
- added R6: 10K, Resistor_SMD:R_0805_2012Metric, F.Cu at (160.0, 121.3)
- added kibuzzard-62D2E07E: G***, kibuzzard-62D2E07E, F.Cu at (113.9, 70.9)
- added kibuzzard-62D2E7EB: G***, kibuzzard-62D2E7EB, F.Cu at (121.9, 78.0)
- added kibuzzard-62D2FEC2: G***, kibuzzard-62D2FEC2, F.Cu at (179.5, 53.6)
- added kibuzzard-62D3EEDE: G***, kibuzzard-62D3EEDE, F.Cu at (198.7, 106.7)
- added kibuzzard-62D3EEF7: G***, kibuzzard-62D3EEF7, F.Cu at (178.3, 117.4)
- added kibuzzard-62D40FBB: G***, kibuzzard-62D40FBB, F.Cu at (163.4, 99.1)
- BZ1: footprint Buzzer_Beeper:Buzzer_12x9.5RM7.6 -> Buzzer_Beeper:MagneticBuzzer_CUI_CST-931RP-A
- moved R7 50.7 mm to (172.8, 104.1), turned to 180 degrees
- moved J5 47.6 mm to (185.5, 106.0)
- moved R9 47.3 mm to (172.8, 106.2), turned to 0 degrees
- moved R10 47.1 mm to (172.8, 115.8), turned to 0 degrees
- moved D4 43.1 mm to (172.8, 108.3)
- moved D5 43.0 mm to (172.8, 113.7)
- moved BZ1 40.8 mm to (152.2, 120.1), turned to 90 degrees
- moved J2 39.9 mm to (180.7, 113.3)
- moved R8 28.9 mm to (130.9, 122.5)
- moved J3 28.5 mm to (161.4, 128.5), turned to 0 degrees
- moved D6 28.2 mm to (122.9, 112.0), turned to -90 degrees
- moved Q1 26.0 mm to (131.7, 126.2), turned to 90 degrees
- moved R12 22.6 mm to (130.9, 119.1)
- moved R11 11.4 mm to (162.0, 121.3), turned to 90 degrees
- moved C7 11.1 mm to (173.3, 111.4), turned to 180 degrees
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- renumbered C8 to C7, D5 to D4, D6 to D5, D4 to D6, R12 to R10, R6 to R11, R7 to R12, R9 to R14, R13 to R15, R14 to R16, R15 to R17, R16 to R18, R17 to R19, R18 to R20, R19 to R21, R20 to R22, R21 to R23, R22 to R24, R23 to R25, R24 to R26, R25 to R27, R26 to R28, R27 to R29, R28 to R30, R29 to R31, R30 to R32, R31 to R33, R32 to R34, R33 to R35, R34 to R36, R35 to R37, R36 to R38, R37 to R39, R38 to R40, R39 to R41, R40 to R42, R41 to R43, R42 to R44, R43 to R45, R44 to R46, R45 to R47, R46 to R48, R47 to R49, R48 to R50, R49 to R51, R50 to R52, R51 to R53, R52 to R54, R53 to R55, R54 to R56, R55 to R57, R56 to R58, R57 to R59, R58 to R60, R59 to R61, R10 to R7, R11 to R9
Connections:
- A1 pad a8: unconnected-(A1-Pada8) -> /_MAIN_SOC/REL3
- J2 pad 2: /_INPUTS/3V3 -> /_MAIN_SOC/5V
- J3 pad 1: /_MAIN_SOC/I2C1_SDA -> GND
- J3 pad 2: /_MAIN_SOC/I2C1_SCK -> /_MAIN_SOC/IOVCC
- J3 pad 3: /_INPUTS/3V3 -> /_MAIN_SOC/I2C1_SCK
- J3 pad 4: GND -> /_MAIN_SOC/I2C1_SDA
- J4 pad 1: /_MAIN_SOC/SPI1_MOSI -> GND
- J4 pad 2: /_MAIN_SOC/SPI1_MISO -> /_MAIN_SOC/IOVCC
- J4 pad 3: /_MAIN_SOC/SPI1_CLK -> /_MAIN_SOC/SPI1_CS
- J4 pad 4: /_MAIN_SOC/SPI1_CS -> /_MAIN_SOC/SPI1_CLK
- J4 pad 5: /_INPUTS/3V3 -> /_MAIN_SOC/SPI1_MISO
- J4 pad 6: GND -> /_MAIN_SOC/SPI1_MOSI
- J5 pad 2: /_INPUTS/3V3 -> /_MAIN_SOC/5V
- Q1 pad 1: /_MAIN_SOC/_BUZZER -> Net-(Q1-Pad1)
- R8 pad 1: /_MAIN_SOC/_BUZZER -> Net-(Q1-Pad1)
Routing:
- net /_MAIN_SOC/5V: track 0.00 -> 202.1 mm, vias 0 -> 3
- net /_INPUTS/3V3: track 29.2 -> 109.7 mm
- net Net-(D30-Pad2): track 0.00 -> 70.0 mm
- net /_MAIN_SOC/REL1: track 0.00 -> 62.3 mm
- net Net-(D28-Pad2): track 0.00 -> 46.1 mm
- net /_MAIN_SOC/REL2: track 0.00 -> 43.8 mm
- net Net-(Q1-Pad1): track 0.00 -> 40.0 mm
- net Net-(D19-Pad2): track 0.00 -> 36.2 mm
- net Net-(BZ1-Pad2): track 0.00 -> 36.0 mm
- net /_MAIN_SOC/I2C0_SDA: track 0.00 -> 35.2 mm
- net /_POWER/12V@2A_ADJ_1: track 9.56 -> 43.8 mm
- net /_MAIN_SOC/SPI1_CLK: track 0.00 -> 33.3 mm
- net /_MAIN_SOC/SPI1_CS: track 0.00 -> 32.7 mm
- net /_MAIN_SOC/SPI1_MISO: track 0.00 -> 32.0 mm
- net /_MAIN_SOC/SPI1_MOSI: track 0.00 -> 31.0 mm
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- added copper zone on F.Cu, net /_POWER/VIN_F
Other:
- board text added: "12~28V"
- board text added: "Designed in Spain Assembled in Lithuania from global materials"
- board text added: "JLCJLCJLCJLC"
- board text removed: "MAGLOCK v2.0 makerspace.lt (Ↄ)2022 Designed in Spain Assembled in Lithuania from global materials"

Commit message: adding more info to silkscreen
Parts:
- added G***: LOGO, -local:qr_maglock_link, B.Cu at (140.0, 115.8)
Routing:
- net GND: track 63.7 -> 78.4 mm, vias 163 -> 162
Other:
- board text added: "+ + - -"
- board text added: "+ - + - + - + -"
- board text added: "3v3"
- board text added: "5v"
- board text added: "GN Vc CS CL MI MO"
- board text added: "GND Vcc SCK SDA"
- board text added: "LOCK"
- board text added: "OUT 2"
- board text added: "OUT 3"
- board text added: "Orange PI zero (plus) goes here"
- board text added: "SDA SCK 5V GND"
- board text added: "SW1"
- board text added: "SW2"
- board text added: "SW3"
- board text added: "SW4"
- board text added: "Vcc"
- board text added: "Vcc SW GND Vcc SW GND Vcc SW GND"
- board text added: "Vin 12~28VDC"

Commit message: adding documentation layers
Parts:
- D13, D14, D15: value RED -> GREEN
- moved J13 5.08 mm to (146.2, 95.2), turned to 180 degrees
- moved J14 5.08 mm to (114.4, 122.7), turned to 180 degrees
- moved J11 5.08 mm to (164.4, 64.3), turned to 180 degrees
- moved J12 5.08 mm to (164.4, 79.8), turned to 180 degrees
- moved J15 5.08 mm to (164.4, 95.1), turned to 180 degrees
- moved kibuzzard-62CDE8D9 0.94 mm to (117.1, 125.8)
Connections:
- J11 pad 1: /_POWER/VOUT4 -> GND
- J11 pad 3: GND -> /_POWER/VOUT4
- J12 pad 1: /_POWER/VOUT5 -> GND
- J12 pad 3: GND -> /_POWER/VOUT5
- J13 pad 1: /_POWER/VOUT1 -> GND
- J13 pad 3: GND -> /_POWER/VOUT1
- J14 pad 1: /_POWER/VOUT2 -> GND
- J14 pad 3: GND -> /_POWER/VOUT2
- J15 pad 1: /_POWER/VOUT3 -> GND
- J15 pad 3: GND -> /_POWER/VOUT3
Routing:
- net /_MAIN_SOC/5V: vias 3 -> 7
Other:
- board text added: "Beeper indicator (Blue)"
- board text added: "Board Dimensions"
- board text added: "Bottom USB Power OK (Red)"
- board text added: "Button Inputs"
- board text added: "Console Power 3v3 OK (Orange)"
- board text added: "Console RX Activity (Green)"
- board text added: "Console TX Activity (Green)"
- board text added: "Display"
- board text added: "Door Close Relay ON (green)"
- board text added: "Door Open Relay ON (green)"
- board text added: "Door PSU 12V Adjust"
- board text added: "Door PSU 12V2 output OK (Yellow) Relays 2 and 3"
- board text added: "Door PSU Fuse (12V2): 2A"
- board text added: "GN D+ D- Vc"
- board text added: "Input Fuse 7A"
- board text added: "Input Power OK (Yellow)"
- board text added: "Input Power Reverse Polatiry (Blue)"
- board text added: "LED Indicators"
- board text added: "Magnet PSU 12V Adjust"
- board text added: "Magnet PSU 12V1 output OK (Yellow) Relay 1"
- board text added: "Magnet PSU Fuse (12V1): 2A"
- board text added: "Magnet Relay ON (green)"
- board text added: "Mounting Holes"
- board text added: "OFF"
- board text added: "ON"
- board text added: "PSU Output"
- board text added: "Power And Fuses"
- board text added: "Power Input and Distribution"
- board text added: "Relay Outputs"
- board text added: "Relay PSU 5V"
- board text added: "Relay PSU 5V3 output OK (Red)"
- board text added: "Relay PSU Fuse (5V3): 1A"
- board text added: "SoC Orange PI zero"
- board text added: "SoC PSU 5V"
- board text added: "SoC PSU 5V1 output OK (Red)"
- board text added: "SoC PSU Fuse (5V1): 1A"
- board text added: "SoC Power 3v3 OK (Orange)"
- board text added: "SoC Power 5v OK (Red)"
- board text added: "Top USB Power OK (Red)"
- board text added: "USB Bottom Port: PTC 300mA"
- board text added: "USB Devices"
- board text added: "USB PSU 5V"
- board text added: "USB PSU 5V2 output OK (Red)"
- board text added: "USB PSU Fuse (5V2): 1A"
- board text added: "USB Top Port: PTC 300mA"
- board text added: "USB UART Debug Conso"

Commit message: adding usb port 3d model
Parts:
- J6: footprint Connector_USB:USB_A_Wuerth_61400826021_Horizontal_Stacked -> -local:USB_A_Wuerth_61400826021_Horizontal_Stacked

Commit message: ERC, DRC and BOM fixes
Parts:
- J7: value Lock -> 3pin
- J8: value Door Open -> 3pin
- J9: value Door Close -> 3pin
- K1, K2, K3: value FINDER-36.11 -> 5V Relay
- R1, R2: value 5k1 -> 4k7
- R11, R12, R13: value 100 -> 330
- R36, R37, R38, R6, R8: value 10K -> 10k

Commit message: bom and documentation fixes
Other:
- board text added: "Functional Overview"
Changed lines of the file:
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@@
     (attr board_only exclude_from_pos_files exclude_from_bom)
     (fp_text reference "kibuzzard-62D3EEDE" (at 0 -4.2926) (layer "F.SilkS") hide
-      (effects (font (size 0 0)))
+      (effects (font (size 0 0) (thickness 0.15)))
     )
     (fp_text value "G***" (at 0 4.2926) (layer "F.SilkS") hide
-      (effects (font (size 0 0)))
+      (effects (font (size 0 0) (thickness 0.15)))
     )
     (fp_poly (pts
@@
     (attr board_only exclude_from_pos_files exclude_from_bom)
     (fp_text reference "kibuzzard-62D2FEC2" (at 0 -4.35696) (layer "F.SilkS") hide
-      (effects (font (size 0 0)))
+      (effects (font (size 0 0) (thickness 0.15)))
     )
     (fp_text value "G***" (at 0 4.35696) (layer "F.SilkS") hide
-      (effects (font (size 0 0)))
+      (effects (font (size 0 0) (thickness 0.15)))
     )
     (fp_poly (pts
@@
     (attr board_only exclude_from_pos_files exclude_from_bom)
     (fp_text reference "kibuzzard-62D40FBB" (at 0 -4.06109 90) (layer "F.SilkS") hide
-      (effects (font (size 0 0)))
+      (effects (font (size 0 0) (thickness 0.15)))
     )
     (fp_text value "G***" (at 0 4.06109 90) (layer "F.SilkS") hide
-      (effects (font (size 0 0)))
+      (effects (font (size 0 0) (thickness 0.15)))
     )
     (fp_poly (pts
@@
     (attr board_only exclude_from_pos_files exclude_from_bom)
     (fp_text reference "kibuzzard-62D2E7EB" (at 0 -4.2926) (layer "F.SilkS") hide
-      (effects (font (size 0 0)))
+      (effects (font (size 0 0) (thickness 0.15)))
     )
     (fp_text value "G***" (at 0 4.2926) (layer "F.SilkS") hide
-      (effects (font (size 0 0)))
+      (effects (font (size 0 0) (thickness 0.15)))
     )
     (fp_poly (pts
@@
     (attr board_only exclude_from_pos_files exclude_from_bom)
     (fp_text reference "kibuzzard-62D2E07E" (at 0 -4.018955 -90) (layer "F.SilkS") hide
-      (effects (font (size 0 0)))
+      (effects (font (size 0 0) (thickness 0.15)))
     )
     (fp_text value "G***" (at 0 4.018955 -90) (layer "F.SilkS") hide
-      (effects (font (size 0 0)))
+      (effects (font (size 0 0) (thickness 0.15)))
     )
     (fp_poly (pts
@@
     (attr board_only exclude_from_pos_files exclude_from_bom)
     (fp_text reference "kibuzzard-62D3EEF7" (at 0 -4.2926) (layer "F.SilkS") hide
-      (effects (font (size 0 0)))
+      (effects (font (size 0 0) (thickness 0.15)))
     )
     (fp_text value "G***" (at 0 4.2926) (layer "F.SilkS") hide
-      (effects (font (size 0 0)))
+      (effects (font (size 0 0) (thickness 0.15)))
     )
     (fp_poly (pts
@@
     (property "Sheetname" "_USB_PORTS")
     (attr through_hole)
-    (fp_text reference "J6" (at 3.5 -3) (layer "F.SilkS")
+    (fp_text reference "J6" (at -4.1 2.53) (layer "F.SilkS")
       (effects (font (size 1 1) (thickness 0.15)))
     )
@@
     (effects (font (size 3 3) (thickness 0.75)))
   )
+  (gr_text "Functional Overview" (at 15 20) (layer "User.2")
+    (effects (font (size 6 6) (thickness 1.5)) (justify left))
+  )
   (gr_text "Relay\nOutputs" (at 184.2 77.7) (layer "User.2")
     (effects (font (size 3 3) (thickness 0.75)))
@@
     (pts (xy 131 150) (xy 131 131))
     (height 8)
-    (gr_text "19.00" (at 135.5 140.5 90) (layer "User.8")
+    (gr_text "19" (at 135.5 140.5 90) (layer "User.8")
       (effects (font (size 3 3) (thickness 0.5)))
     )
-    (format (units 3) (units_format 0) (precision 2))
+    (format (units 2) (units_format 0) (precision 2) suppress_zeroes)
     (style (thickness 0.15) (arrow_length 1.27) (text_position_mode 0) (extension_height 0.58642) (extension_offset 0.5) keep_text_aligned)
   )
@@
     (pts (xy 109 150) (xy 109 52))
     (height -14)
-    (gr_text "98.00" (at 91.5 101 90) (layer "User.8")
+    (gr_text "98" (at 91.5 101 90) (layer "User.8")
       (effects (font (size 3 3) (thickness 0.5)))
     )
-    (format (units 3) (units_format 0) (precision 2))
+    (format (units 2) (units_format 0) (precision 2) suppress_zeroes)
     (style (thickness 0.15) (arrow_length 1.27) (text_position_mode 0) (extension_height 0.58642) (extension_offset 0.5) keep_text_aligned)
   )
@@
     (pts (xy 130 146) (xy 105 146))
     (height -24)
-    (gr_text "25.00" (at 117.5 166.5) (layer "User.8")
+    (gr_text "25" (at 117.5 166.5) (layer "User.8")
       (effects (font (size 3 3) (thickness 0.5)))
     )
-    (format (units 3) (units_format 0) (precision 2))
+    (format (units 2) (units_format 0) (precision 2) suppress_zeroes)
     (style (thickness 0.15) (arrow_length 1.27) (text_position_mode 0) (extension_height 0.58642) (extension_offset 0.5) keep_text_aligned)
   )
@@
     (pts (xy 203 56) (xy 105 56))
     (height 16)
-    (gr_text "98.00" (at 154 36.5) (layer "User.8")
+    (gr_text "98" (at 154 36.5) (layer "User.8")
       (effects (font (size 3 3) (thickness 0.5)))
     )
-    (format (units 3) (units_format 0) (precision 2))
+    (format (units 2) (units_format 0) (precision 2) suppress_zeroes)
     (style (thickness 0.15) (arrow_length 1.27) (text_position_mode 0) (extension_height 0.58642) (extension_offset 0.5) keep_text_aligned)
   )
@@
     (pts (xy 157 146) (xy 130 146))
     (height -24)
-    (gr_text "27.00" (at 143.5 166.5) (layer "User.8")
+    (gr_text "27" (at 143.5 166.5) (layer "User.8")
       (effects (font (size 3 3) (thickness 0.5)))
     )
-    (format (units 3) (units_format 0) (precision 2))
+    (format (units 2) (units_format 0) (precision 2) suppress_zeroes)
     (style (thickness 0.15) (arrow_length 1.27) (text_position_mode 0) (extension_height 0.58642) (extension_offset 0.5) keep_text_aligned)
   )
@@
       (effects (font (size 3 3) (thickness 0.5)))
     )
-    (format (units 3) (units_format 0) (precision 2) suppress_zeroes)
+    (format (units 2) (units_format 0) (precision 2) suppress_zeroes)
     (style (thickness 0.15) (arrow_length 1.27) (text_position_mode 2) (extension_height 0.58642) (extension_offset 0.5) keep_text_aligned)
   )
@@
       (effects (font (size 3 3) (thickness 0.5)))
     )
-    (format (units 3) (units_format 0) (precision 2) suppress_zeroes)
+    (format (units 2) (units_format 0) (precision 2) suppress_zeroes)
     (style (thickness 0.15) (arrow_length 1.27) (text_position_mode 0) (extension_height 0.58642) (extension_offset 0.5) keep_text_aligned)
   )
@@
       (effects (font (size 3 3) (thickness 0.5)))
     )
-    (format (units 3) (units_format 0) (precision 2) suppress_zeroes)
+    (format (units 2) (units_format 0) (precision 2) suppress_zeroes)
     (style (thickness 0.15) (arrow_length 1.27) (text_position_mode 0) (extension_height 0.58642) (extension_offset 0.5) keep_text_aligned)
   )
@@
       (effects (font (size 3 3) (thickness 0.5)))
     )
-    (format (units 3) (units_format 0) (precision 2) suppress_zeroes)
+    (format (units 2) (units_format 0) (precision 2) suppress_zeroes)
     (style (thickness 0.15) (arrow_length 1.27) (text_position_mode 0) (extension_height 0.58642) (extension_offset 0.5) keep_text_aligned)
   )
@@
       (effects (font (size 3 3) (thickness 0.5)))
     )
-    (format (units 3) (units_format 0) (precision 2) suppress_zeroes)
+    (format (units 2) (units_format 0) (precision 2) suppress_zeroes)
     (style (thickness 0.15) (arrow_length 1.27) (text_position_mode 0) (extension_height 0.58642) (extension_offset 0.5) keep_text_aligned)
   )
@@
       (effects (font (size 3 3) (thickness 0.5)))
     )
-    (format (units 3) (units_format 0) (precision 2) suppress_zeroes)
+    (format (units 2) (units_format 0) (precision 2) suppress_zeroes)
     (style (thickness 0.15) (arrow_length 1.27) (text_position_mode 0) (extension_height 0.58642) (extension_offset 0.5) keep_text_aligned)
   )
@@
       (effects (font (size 3 3) (thickness 0.5)))
     )
-    (format (units 3) (units_format 0) (precision 2) suppress_zeroes)
+    (format (units 2) (units_format 0) (precision 2) suppress_zeroes)
     (style (thickness 0.15) (arrow_length 1.27) (text_position_mode 0) (extension_height 0.58642) (extension_offset 0.5) keep_text_aligned)
   )
@@
       (effects (font (size 3 3) (thickness 0.5)))
     )
-    (format (units 3) (units_format 0) (precision 2) suppress_zeroes)
+    (format (units 2) (units_format 0) (precision 2) suppress_zeroes)
     (style (thickness 0.15) (arrow_length 1.27) (text_position_mode 0) (extension_height 0.58642) (extension_offset 0.5) keep_text_aligned)
   )
