File: maglock.kicad_pcb (KiCad board)
At the start: 2 copper layers, 98 x 98 mm, 222 parts, among them J1 USB_UART, J10 Power IN, J11 12V_1, J12 12V_2, J13 5V_1, J14 5V_2, J15 5V_3, J2 I2C0_128x32, J3 I2C1, J4 SPI1, J5 I2C0_128x64, J6 USB, J7 3pin, J8 3pin, J9 3pin, K1 5V Relay, K2 5V Relay, K3 5V Relay, Q1 AO3400A, Q2 AO3400A, Q3 AO3400A, Q4 AO3400A, Q5 HYG210P06LQ1D, SW1 2pin, SW2 2pin, SW3 2pin, SW4 2pin, U1 USBLC6-2SC6, U10 XL4001, U11 XL4001, U2 3V3 LDO, U3 CH340C, U4 DS18B20Z, U5 USBLC6-2SC6, U6 USBLC6-2SC6, U7 XL4001, U8 XL4001, U9 XL4001

Commit message: updating qr link to include version
Parts:
- moved G*** 1.12 mm to (140.2, 114.7)
Other:
- board text added: "ID:"
- board text added: "S/N:"

Commit message: adding pre/post release checklist and preparing for fixes
Parts:
- removed kibuzzard-62D3EEDE: G***, kibuzzard-62D3EEDE
- added kibuzzard-636121EB: G***, kibuzzard-636121EB, F.Cu at (198.7, 106.7)

Commit message: adding direction markers for pots. fixes #2
Parts:
- RV1, RV2: footprint Potentiometer_THT:Potentiometer_Bourns_3296W_Vertical -> -local:Potentiometer_Bourns_3296W_Vertical
- moved LOGO1 0.09 mm to (124.8, 83.3)

Commit message: adding direction marker for buzzer. fixes #4
Parts:
- BZ1: footprint Buzzer_Beeper:MagneticBuzzer_CUI_CST-931RP-A -> -local:MagneticBuzzer_CUI_CST-931RP-A
Changed lines of the file:
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@@
     )
   )
-  (footprint "Buzzer_Beeper:MagneticBuzzer_CUI_CST-931RP-A" (layer "F.Cu")
+  (footprint "-local:MagneticBuzzer_CUI_CST-931RP-A" (layer "F.Cu")
     (at 152.168 120.087 90)
     (descr "CST-931RP-A, http://www.cui.com/product/resource/cst-931rp-a.pdf")
@@
       (effects (font (size 1 1) (thickness 0.15)))
     )
+    (fp_text user "${REFERENCE}" (at 0 2 90) (layer "F.Fab")
+      (effects (font (size 1 1) (thickness 0.15)))
+    )
     (fp_text user "+" (at -1.5 -0.1 90) (layer "F.Fab")
       (effects (font (size 1 1) (thickness 0.15)))
     )
-    (fp_text user "${REFERENCE}" (at 0 2 90) (layer "F.Fab")
-      (effects (font (size 1 1) (thickness 0.15)))
-    )
+    (fp_line (start 2.54 -4.064) (end 2.54 -1.905) (layer "F.SilkS") (width 0.12))
+    (fp_line (start -2.54 -1.905) (end -2.54 -4.064) (layer "F.SilkS") (width 0.12))
+    (fp_line (start -2.54 -4.064) (end 2.54 -4.064) (layer "F.SilkS") (width 0.12))
     (fp_circle (center 0 2) (end 4.62 2) (layer "F.SilkS") (width 0.12) (fill none))
+    (fp_line (start -2.75 -1.88) (end -2.75 -4.25) (layer "F.CrtYd") (width 0.05))
     (fp_line (start -2.75 -4.25) (end 2.75 -4.25) (layer "F.CrtYd") (width 0.05))
-    (fp_line (start -2.75 -1.88) (end -2.75 -4.25) (layer "F.CrtYd") (width 0.05))
     (fp_line (start 2.75 -4.25) (end 2.75 -1.88) (layer "F.CrtYd") (width 0.05))
     (fp_arc (start 2.75 -1.88) (mid 0.006009 6.755719) (end -2.759797 -1.873038) (layer "F.CrtYd") (width 0.05))
     (fp_line (start -2.5 -4) (end -2.5 -1.74) (layer "F.Fab") (width 0.1))
+    (fp_line (start 2.5 -4) (end 2.5 -1.74) (layer "F.Fab") (width 0.1))
     (fp_line (start -2.5 -4) (end 2.5 -4) (layer "F.Fab") (width 0.1))
-    (fp_line (start 2.5 -4) (end 2.5 -1.74) (layer "F.Fab") (width 0.1))
     (fp_arc (start 2.5 -1.74) (mid 0.003084 6.498621) (end -2.505126 -1.736568) (layer "F.Fab") (width 0.1))
     (pad "1" thru_hole rect (at 0 0 90) (size 1.6 1.6) (drill 0.9) (layers *.Cu *.Mask)
