File: maglock.kicad_pcb (KiCad board)
At the start: 2 copper layers, 98 x 98 mm, 222 parts, among them J1 USB_UART, J10 Power IN, J11 12V_1, J12 12V_2, J13 5V_1, J14 5V_2, J15 5V_3, J2 I2C0_128x32, J3 I2C1, J4 SPI1, J5 I2C0_128x64, J6 USB, J7 3pin, J8 3pin, J9 3pin, K1 5V Relay, K2 5V Relay, K3 5V Relay, Q1 AO3400A, Q2 AO3400A, Q3 AO3400A, Q4 AO3400A, Q5 HYG210P06LQ1D, SW1 2pin, SW2 2pin, SW3 2pin, SW4 2pin, U1 USBLC6-2SC6, U10 XL4001, U11 XL4001, U2 3V3 LDO, U3 CH340C, U4 DS18B20Z, U5 USBLC6-2SC6, U6 USBLC6-2SC6, U7 XL4001, U8 XL4001, U9 XL4001

Commit message: removing unreadable text from OSHW logo. fixes #15
Parts:
- LOGO2: footprint Symbol:OSHW-Logo2_9.8x8mm_SilkScreen -> Symbol:OSHW-Symbol_6.7x6mm_SilkScreen
- moved LOGO2 0.80 mm to (117.7, 83.2)

Commit message: fixing hole spacing in the buzzer footprint. fixes #3
Parts:
- R11: value 330 -> 0
- R15, R17, R19, R21: value 10k -> 0
- R31, R32: value 330 -> 4k7
- R44: value 100k -> 10k
- R59, R60, R61: value 1k -> 4k7
- moved BZ1 0.42 mm to (151.7, 120.1)
Changed lines of the file:
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@@
       (effects (font (size 1 1) (thickness 0.15)))
     )
-    (fp_text value "1k" (at 0 1.65 90) (layer "F.Fab")
+    (fp_text value "4k7" (at 0 1.65 90) (layer "F.Fab")
       (effects (font (size 1 1) (thickness 0.15)))
     )
@@
       (effects (font (size 1 1) (thickness 0.15)))
     )
-    (fp_text value "330" (at 0 1.65 90) (layer "F.Fab")
+    (fp_text value "4k7" (at 0 1.65 90) (layer "F.Fab")
       (effects (font (size 1 1) (thickness 0.15)))
     )
@@
       (effects (font (size 1 1) (thickness 0.15)))
     )
-    (fp_text value "10k" (at 0 1.65) (layer "F.Fab")
+    (fp_text value "0" (at 0 1.65) (layer "F.Fab")
       (effects (font (size 1 1) (thickness 0.15)))
     )
@@
       (effects (font (size 1 1) (thickness 0.15)))
     )
-    (fp_text value "330" (at 0 1.65 90) (layer "F.Fab")
+    (fp_text value "0" (at 0 1.65 90) (layer "F.Fab")
       (effects (font (size 1 1) (thickness 0.15)))
     )
@@
       (effects (font (size 1 1) (thickness 0.15)))
     )
-    (fp_text value "100k" (at 0 1.65) (layer "F.Fab")
+    (fp_text value "10k" (at 0 1.65) (layer "F.Fab")
       (effects (font (size 1 1) (thickness 0.15)))
     )
@@
       (effects (font (size 1 1) (thickness 0.15)))
     )
-    (fp_text value "330" (at 0 1.65 90) (layer "F.Fab")
+    (fp_text value "4k7" (at 0 1.65 90) (layer "F.Fab")
       (effects (font (size 1 1) (thickness 0.15)))
     )
@@
       (effects (font (size 1 1) (thickness 0.15)))
     )
-    (fp_text value "10k" (at 0 1.65) (layer "F.Fab")
+    (fp_text value "0" (at 0 1.65) (layer "F.Fab")
       (effects (font (size 1 1) (thickness 0.15)))
     )
@@
       (effects (font (size 1 1) (thickness 0.15)))
     )
-    (fp_text value "1k" (at 0 1.65) (layer "F.Fab")
+    (fp_text value "4k7" (at 0 1.65) (layer "F.Fab")
       (effects (font (size 1 1) (thickness 0.15)))
     )
@@
       (effects (font (size 1 1) (thickness 0.15)))
     )
-    (fp_text value "10k" (at 0 1.65) (layer "F.Fab")
+    (fp_text value "0" (at 0 1.65) (layer "F.Fab")
       (effects (font (size 1 1) (thickness 0.15)))
     )
@@
   )
   (footprint "-local:MagneticBuzzer_CUI_CST-931RP-A" (layer "F.Cu")
-    (at 152.168 120.087 90)
+    (at 151.747139 120.087 90)
     (descr "CST-931RP-A, http://www.cui.com/product/resource/cst-931rp-a.pdf")
     (tags "CST-931RP-A")
@@
       (effects (font (size 1 1) (thickness 0.15)))
     )
-    (fp_text user "${REFERENCE}" (at 0 2 90) (layer "F.Fab")
+    (fp_text user "+" (at -1.5 -0.1 90) (layer "F.Fab")
       (effects (font (size 1 1) (thickness 0.15)))
     )
-    (fp_text user "+" (at -1.5 -0.1 90) (layer "F.Fab")
+    (fp_text user "${REFERENCE}" (at 0 2 90) (layer "F.Fab")
       (effects (font (size 1 1) (thickness 0.15)))
     )
-    (fp_line (start 2.54 -4.064) (end 2.54 -1.905) (layer "F.SilkS") (width 0.12))
-    (fp_line (start -2.54 -1.905) (end -2.54 -4.064) (layer "F.SilkS") (width 0.12))
-    (fp_line (start -2.54 -4.064) (end 2.54 -4.064) (layer "F.SilkS") (width 0.12))
-    (fp_circle (center 0 2) (end 4.62 2) (layer "F.SilkS") (width 0.12) (fill none))
-    (fp_line (start -2.75 -1.88) (end -2.75 -4.25) (layer "F.CrtYd") (width 0.05))
-    (fp_line (start -2.75 -4.25) (end 2.75 -4.25) (layer "F.CrtYd") (width 0.05))
-    (fp_line (start 2.75 -4.25) (end 2.75 -1.88) (layer "F.CrtYd") (width 0.05))
-    (fp_arc (start 2.75 -1.88) (mid 0.006009 6.755719) (end -2.759797 -1.873038) (layer "F.CrtYd") (width 0.05))
-    (fp_line (start -2.5 -4) (end -2.5 -1.74) (layer "F.Fab") (width 0.1))
-    (fp_line (start 2.5 -4) (end 2.5 -1.74) (layer "F.Fab") (width 0.1))
-    (fp_line (start -2.5 -4) (end 2.5 -4) (layer "F.Fab") (width 0.1))
-    (fp_arc (start 2.5 -1.74) (mid 0.003084 6.498621) (end -2.505126 -1.736568) (layer "F.Fab") (width 0.1))
+    (fp_line (start 2.54 -3.564) (end 2.54 -1.405) (layer "F.SilkS") (width 0.12))
+    (fp_line (start -2.54 -1.405) (end -2.54 -3.564) (layer "F.SilkS") (width 0.12))
+    (fp_line (start -2.54 -3.564) (end 2.54 -3.564) (layer "F.SilkS") (width 0.12))
+    (fp_circle (center 0 2.5) (end 4.62 2.5) (layer "F.SilkS") (width 0.12) (fill none))
+    (fp_line (start 2.75 -3.75) (end 2.75 -1.38) (layer "F.CrtYd") (width 0.05))
+    (fp_line (start -2.75 -3.75) (end 2.75 -3.75) (layer "F.CrtYd") (width 0.05))
+    (fp_line (start -2.75 -1.38) (end -2.75 -3.75) (layer "F.CrtYd") (width 0.05))
+    (fp_arc (start 2.75 -1.38) (mid 0.006009 7.255719) (end -2.759797 -1.373038) (layer "F.CrtYd") (width 0.05))
+    (fp_line (start 2.5 -3.5) (end 2.5 -1.24) (layer "F.Fab") (width 0.1))
+    (fp_line (start -2.5 -3.5) (end -2.5 -1.24) (layer "F.Fab") (width 0.1))
+    (fp_line (start -2.5 -3.5) (end 2.5 -3.5) (layer "F.Fab") (width 0.1))
+    (fp_arc (start 2.5 -1.24) (mid 0.003084 6.998621) (end -2.505126 -1.236568) (layer "F.Fab") (width 0.1))
     (pad "1" thru_hole rect (at 0 0 90) (size 1.6 1.6) (drill 0.9) (layers *.Cu *.Mask)
       (net 57 "Net-(BZ1-Pad1)") (pinfunction "-") (pintype "passive"))
-    (pad "2" thru_hole circle (at 0 4 90) (size 1.6 1.6) (drill 0.9) (layers *.Cu *.Mask)
+    (pad "2" thru_hole circle (at 0 5 90) (size 1.6 1.6) (drill 0.9) (layers *.Cu *.Mask)
       (net 56 "Net-(BZ1-Pad2)") (pinfunction "+") (pintype "passive"))
     (model "${KICAD6_3DMODEL_DIR}/Buzzer_Beeper.3dshapes/MagneticBuzzer_CUI_CST-931RP-A.wrl"
-      (offset (xyz 0 0 0))
+      (offset (xyz 0 -0.5 0))
       (scale (xyz 1 1 1))
       (rotate (xyz 0 0 0))
@@
       (effects (font (size 1 1) (thickness 0.15)))
     )
-    (fp_text value "1k" (at 0 1.65) (layer "F.Fab")
+    (fp_text value "4k7" (at 0 1.65) (layer "F.Fab")
       (effects (font (size 1 1) (thickness 0.15)))
     )
@@
       (effects (font (size 1 1) (thickness 0.15)))
     )
-    (fp_text value "10k" (at 0 1.65) (layer "F.Fab")
+    (fp_text value "0" (at 0 1.65) (layer "F.Fab")
       (effects (font (size 1 1) (thickness 0.15)))
     )

Commit message: removing an unnecessary resistor from OPI 5V indicator. fixes #6
Parts:
- removed R9: 1k, Resistor_SMD:R_0805_2012Metric
- R7: value 1k -> 4k7
- moved R7 2.10 mm to (172.8, 106.2), turned to 0 degrees
Connections:
- R7 pad 2: Net-(R7-Pad2) -> Net-(D4-Pad1)
Routing:
- net Net-(R7-Pad2): track 2.10 -> 0.00 mm
Changed lines of the file:
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@@
   (net 140 "Net-(R45-Pad1)")
   (net 141 "/_MAIN_SOC/IOVCC")
-  (net 142 "Net-(R7-Pad2)")
   (footprint "Resistor_SMD:R_0805_2012Metric" locked (layer "F.Cu")
     (at 107 117.8 90)
@@
       (net 1 "GND") (pinfunction "1") (pintype "input"))
   )
-  (footprint "Resistor_SMD:R_0805_2012Metric" (layer "F.Cu")
-    (at 172.8 106.2)
-    (descr "Resistor SMD 0805 (2012 Metric), square (rectangular) end terminal, IPC_7351 nominal, (Body size source: IPC-SM-782 page 72, https://www.pcb-3d.com/wordpress/wp-content/uploads/ipc-sm-782a_amendment_1_and_2.pdf), generated with kicad-footprint-generator")
-    (tags "resistor")
-    (property "LCSC Part Number" "")
-    (property "Sheetfile" "File: _main_soc.kicad_sch")
-    (property "Sheetname" "_MAIN_SOC")
-    (attr smd)
-    (fp_text reference "R9" (at 2.3 0 90) (layer "F.SilkS")
-      (effects (font (size 1 1) (thickness 0.15)))
-    )
-    (fp_text value "1k" (at 0 1.65) (layer "F.Fab")
-      (effects (font (size 1 1) (thickness 0.15)))
-    )
-    (fp_text user "${REFERENCE}" (at 0 0) (layer "F.Fab")
-      (effects (font (size 0.5 0.5) (thickness 0.08)))
-    )
-    (fp_line (start -0.227064 0.735) (end 0.227064 0.735) (layer "F.SilkS") (width 0.12))
-    (fp_line (start -0.227064 -0.735) (end 0.227064 -0.735) (layer "F.SilkS") (width 0.12))
-    (fp_line (start 1.68 0.95) (end -1.68 0.95) (layer "F.CrtYd") (width 0.05))
-    (fp_line (start -1.68 -0.95) (end 1.68 -0.95) (layer "F.CrtYd") (width 0.05))
-    (fp_line (start -1.68 0.95) (end -1.68 -0.95) (layer "F.CrtYd") (width 0.05))
-    (fp_line (start 1.68 -0.95) (end 1.68 0.95) (layer "F.CrtYd") (width 0.05))
-    (fp_line (start 1 0.625) (end -1 0.625) (layer "F.Fab") (width 0.1))
-    (fp_line (start 1 -0.625) (end 1 0.625) (layer "F.Fab") (width 0.1))
-    (fp_line (start -1 -0.625) (end 1 -0.625) (layer "F.Fab") (width 0.1))
-    (fp_line (start -1 0.625) (end -1 -0.625) (layer "F.Fab") (width 0.1))
-    (pad "1" smd roundrect (at -0.9125 0) (size 1.025 1.4) (layers "F.Cu" "F.Paste" "F.Mask") (roundrect_rratio 0.243902)
-      (net 142 "Net-(R7-Pad2)") (pintype "passive"))
-    (pad "2" smd roundrect (at 0.9125 0) (size 1.025 1.4) (layers "F.Cu" "F.Paste" "F.Mask") (roundrect_rratio 0.243902)
-      (net 65 "Net-(D4-Pad1)") (pintype "passive"))
-    (model "${KICAD6_3DMODEL_DIR}/Resistor_SMD.3dshapes/R_0805_2012Metric.wrl"
-      (offset (xyz 0 0 0))
-      (scale (xyz 1 1 1))
-      (rotate (xyz 0 0 0))
-    )
-  )
   (footprint "Package_SO:Texas_HTSOP-8-1EP_3.9x4.9mm_P1.27mm_EP2.95x4.9mm_Mask2.4x3.1mm_ThermalVias" locked (layer "F.Cu")
     (at 112.67 96.2 90)
@@
   )
   (footprint "Resistor_SMD:R_0805_2012Metric" (layer "F.Cu")
-    (at 172.8 104.1 180)
+    (at 172.8 106.2)
     (descr "Resistor SMD 0805 (2012 Metric), square (rectangular) end terminal, IPC_7351 nominal, (Body size source: IPC-SM-782 page 72, https://www.pcb-3d.com/wordpress/wp-content/uploads/ipc-sm-782a_amendment_1_and_2.pdf), generated with kicad-footprint-generator")
     (tags "resistor")
@@
     (property "Sheetname" "_MAIN_SOC")
     (attr smd)
-    (fp_text reference "R7" (at -2.3 0 90) (layer "F.SilkS")
+    (fp_text reference "R7" (at 0 -1.6 180) (layer "F.SilkS")
       (effects (font (size 1 1) (thickness 0.15)))
     )
-    (fp_text value "1k" (at 0 1.65) (layer "F.Fab")
+    (fp_text value "4k7" (at 0 1.65) (layer "F.Fab")
       (effects (font (size 1 1) (thickness 0.15)))
     )
@@
     (fp_line (start -1 -0.625) (end 1 -0.625) (layer "F.Fab") (width 0.1))
     (fp_line (start 1 0.625) (end -1 0.625) (layer "F.Fab") (width 0.1))
-    (pad "1" smd roundrect (at -0.9125 0 180) (size 1.025 1.4) (layers "F.Cu" "F.Paste" "F.Mask") (roundrect_rratio 0.243902)
+    (pad "1" smd roundrect (at -0.9125 0) (size 1.025 1.4) (layers "F.Cu" "F.Paste" "F.Mask") (roundrect_rratio 0.243902)
       (net 1 "GND") (pintype "passive"))
-    (pad "2" smd roundrect (at 0.9125 0 180) (size 1.025 1.4) (layers "F.Cu" "F.Paste" "F.Mask") (roundrect_rratio 0.243902)
-      (net 142 "Net-(R7-Pad2)") (pintype "passive"))
+    (pad "2" smd roundrect (at 0.9125 0) (size 1.025 1.4) (layers "F.Cu" "F.Paste" "F.Mask") (roundrect_rratio 0.243902)
+      (net 65 "Net-(D4-Pad1)") (pintype "passive"))
     (model "${KICAD6_3DMODEL_DIR}/Resistor_SMD.3dshapes/R_0805_2012Metric.wrl"
       (offset (xyz 0 0 0))
@@
     (property "Sheetname" "_MAIN_SOC")
     (attr through_hole)
-    (fp_text reference "J2" (at 0 -2.18) (layer "F.SilkS")
+    (fp_text reference "J2" (at -2.3 5.08) (layer "F.SilkS")
       (effects (font (size 1 1) (thickness 0.15)))
     )
@@
     (property "WE" "885012108012")
     (attr smd)
-    (fp_text reference "C7" (at -2.3 1.7) (layer "F.SilkS")
+    (fp_text reference "C7" (at -2.9 0 90) (layer "F.SilkS")
       (effects (font (size 1 1) (thickness 0.15)))
     )
@@
     (property "Sheetname" "_MAIN_SOC")
     (attr through_hole)
-    (fp_text reference "J5" (at -1.8 -2 180) (layer "F.SilkS")
+    (fp_text reference "J5" (at 2.2 3.5 180) (layer "F.SilkS")
       (effects (font (size 1 1) (thickness 0.15)))
     )
@@
   (via locked (at 161.1 103.5) (size 0.8) (drill 0.4) (layers "F.Cu" "B.Cu") (net 1))
   (via locked (at 152.5 104.5) (size 0.8) (drill 0.4) (layers "F.Cu" "B.Cu") (net 1))
-  (via (at 173.7 104.1) (size 0.8) (drill 0.4) (layers "F.Cu" "B.Cu") (net 1))
   (via locked (at 154.1 110.5) (size 0.8) (drill 0.4) (layers "F.Cu" "B.Cu") (net 1))
   (via locked (at 115.3 131.4) (size 0.8) (drill 0.4) (layers "F.Cu" "B.Cu") (net 1))
@@
   (via locked (at 121.6 131.1) (size 0.8) (drill 0.4) (layers "F.Cu" "B.Cu") (net 1))
   (via (at 163.8 116) (size 0.8) (drill 0.4) (layers "F.Cu" "B.Cu") (net 1))
+  (via (at 171.8 106.2) (size 0.8) (drill 0.4) (layers "F.Cu" "B.Cu") (net 1))
   (via locked (at 131.85 102.55) (size 0.8) (drill 0.4) (layers "F.Cu" "B.Cu") (net 1))
   (via locked (at 119.4 95) (size 0.8) (drill 0.4) (layers "F.Cu" "B.Cu") (net 1))
@@
   (segment locked (start 183.19952 122.57952) (end 183.19952 128.16798) (width 0.4) (layer "F.Cu") (net 64))
   (segment locked (start 176.34404 121.65596) (end 182.27596 121.65596) (width 0.4) (layer "F.Cu") (net 64))
-  (segment (start 173.825 108.3) (end 173.825 106.3125) (width 0.4) (layer "F.Cu") (net 65))
   (segment (start 173.825 106.3125) (end 173.7125 106.2) (width 0.4) (layer "F.Cu") (net 65))
+  (segment (start 173.825 108.3) (end 173.825 106.3125) (width 0.4) (layer "F.Cu") (net 65))
   (segment (start 173.825 115.6875) (end 173.7125 115.8) (width 0.4) (layer "F.Cu") (net 66))
   (segment (start 173.825 113.7) (end 173.825 115.6875) (width 0.4) (layer "F.Cu") (net 66))
@@
   (segment (start 152.3526 125.387) (end 154.5526 127.587) (width 0.8) (layer "F.Cu") (net 141))
   (segment (start 141.768 125.387) (end 152.3526 125.387) (width 0.8) (layer "F.Cu") (net 141))
-  (segment (start 171.8875 104.1) (end 171.8875 106.2) (width 0.4) (layer "F.Cu") (net 142))
   (zone locked (net 45) (net_name "/_POWER/VIN2") (layer "F.Cu") (hatch edge 0.508)
     (priority 5)

Commit message: improving lx4001 footprint thermals. fixes #7
Parts:
- U10, U11, U7, U8, U9: footprint Package_SO:Texas_HTSOP-8-1EP_3.9x4.9mm_P1.27mm_EP2.95x4.9mm_Mask2.4x3.1mm_ThermalVias -> -local:Texas_HTSOP-8-1EP_3.9x4.9mm_P1.27mm_EP2.8x4.1mm_Mask2.8x4.1mm_ThermalVias

Commit message: fixing Q5 footprint and rerouting. fixes #1
Parts:
- D10, D24, D7, D8, D9: value 3V3 -> 10V
- moved R44 8.22 mm to (121.2, 58.2), turned to 0 degrees
- moved C21 7.05 mm to (121.2, 56.2), turned to 180 degrees
- moved D24 6.40 mm to (121.7, 61.6)
- moved Q5 3.61 mm to (126.5, 58.0), turned to 90 degrees
Connections:
- Q5 pad 2: /_POWER/VIN -> /_POWER/VIN_F
- Q5 pad 3: /_POWER/VIN_F -> /_POWER/VIN
Routing:
- net /_POWER/VIN: track 44.7 -> 48.4 mm
- net /_POWER/VIN_F: track 0.00 -> 2.50 mm
- net Net-(C21-Pad1): track 6.31 -> 7.39 mm
- net GND: vias 162 -> 176
