File: _power.kicad_sch (KiCad schematic)
At the start: 96 parts, among them J10 Power IN, J11 12V_1, J12 12V_2, J13 5V_1, J14 5V_2, J15 5V_3, Q5 HYG210P06LQ1D, U10 XL4001, U11 XL4001, U7 XL4001, U8 XL4001, U9 XL4001

Commit message: driving Q5 harder by decreasing R44 resistance. fixes #14
Parts:
- R44: value 100k -> 10k
Changed lines of the file:
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@@
       (effects (font (size 1.27 1.27)) (justify left))
     )
-    (property "Value" "100k" (id 1) (at 96.52 49.53 90)
+    (property "Value" "10k" (id 1) (at 96.52 50.8 90)
       (effects (font (size 1.27 1.27)) (justify left))
     )

Commit message: reducing PSU and USB power LEDs brightness. fixes #5
Parts:
- R59, R60, R61: value 1k -> 4k7
Changed lines of the file:
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@@
       (effects (font (size 1.27 1.27)) (justify left))
     )
-    (property "Value" "1k" (id 1) (at 261.62 129.54 90)
+    (property "Value" "4k7" (id 1) (at 261.62 129.54 90)
       (effects (font (size 1.27 1.27)) (justify left))
     )
@@
       (effects (font (size 1.27 1.27)) (justify left))
     )
-    (property "Value" "1k" (id 1) (at 261.62 53.34 90)
+    (property "Value" "4k7" (id 1) (at 261.62 53.34 90)
       (effects (font (size 1.27 1.27)) (justify left))
     )
@@
       (effects (font (size 1.27 1.27)) (justify left))
     )
-    (property "Value" "1k" (id 1) (at 261.62 91.44 90)
-      (effects (font (size 1.27 1.27)) (justify left))
-    )
+    (property "Value" "4k7" (id 1) (at 261.62 91.44 90)
+      (effects (font (size 1.27 1.27)) (justify left))
+    )

Commit message: improving lx4001 footprint thermals. fixes #7
Parts:
- U10, U11, U7, U8, U9: footprint Package_SO:Texas_HTSOP-8-1EP_3.9x4.9mm_P1.27mm_EP2.95x4.9mm_Mask2.4x3.1mm_ThermalVias -> -local:Texas_HTSOP-8-1EP_3.9x4.9mm_P1.27mm_EP2.8x4.1mm_Mask2.8x4.1mm_ThermalVias
Changed lines of the file:
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@@
     (property "Reference" "U10" (id 0) (at 205.74 73.66 0))
     (property "Value" "XL4001" (id 1) (at 209.55 86.36 0))
-    (property "Footprint" "Package_SO:Texas_HTSOP-8-1EP_3.9x4.9mm_P1.27mm_EP2.95x4.9mm_Mask2.4x3.1mm_ThermalVias" (id 2) (at 209.55 83.82 0)
+    (property "Footprint" "-local:Texas_HTSOP-8-1EP_3.9x4.9mm_P1.27mm_EP2.8x4.1mm_Mask2.8x4.1mm_ThermalVias" (id 2) (at 209.55 83.82 0)
       (effects (font (size 1.27 1.27)) hide)
     )
@@
     (property "Reference" "U9" (id 0) (at 205.74 35.56 0))
     (property "Value" "XL4001" (id 1) (at 209.55 48.26 0))
-    (property "Footprint" "Package_SO:Texas_HTSOP-8-1EP_3.9x4.9mm_P1.27mm_EP2.95x4.9mm_Mask2.4x3.1mm_ThermalVias" (id 2) (at 209.55 45.72 0)
+    (property "Footprint" "-local:Texas_HTSOP-8-1EP_3.9x4.9mm_P1.27mm_EP2.8x4.1mm_Mask2.8x4.1mm_ThermalVias" (id 2) (at 209.55 45.72 0)
       (effects (font (size 1.27 1.27)) hide)
     )
@@
     (property "Reference" "U8" (id 0) (at 66.04 111.76 0))
     (property "Value" "XL4001" (id 1) (at 69.85 124.46 0))
-    (property "Footprint" "Package_SO:Texas_HTSOP-8-1EP_3.9x4.9mm_P1.27mm_EP2.95x4.9mm_Mask2.4x3.1mm_ThermalVias" (id 2) (at 69.85 121.92 0)
+    (property "Footprint" "-local:Texas_HTSOP-8-1EP_3.9x4.9mm_P1.27mm_EP2.8x4.1mm_Mask2.8x4.1mm_ThermalVias" (id 2) (at 69.85 121.92 0)
       (effects (font (size 1.27 1.27)) hide)
     )
@@
     (property "Reference" "U11" (id 0) (at 205.74 111.76 0))
     (property "Value" "XL4001" (id 1) (at 209.55 124.46 0))
-    (property "Footprint" "Package_SO:Texas_HTSOP-8-1EP_3.9x4.9mm_P1.27mm_EP2.95x4.9mm_Mask2.4x3.1mm_ThermalVias" (id 2) (at 209.55 121.92 0)
+    (property "Footprint" "-local:Texas_HTSOP-8-1EP_3.9x4.9mm_P1.27mm_EP2.8x4.1mm_Mask2.8x4.1mm_ThermalVias" (id 2) (at 209.55 121.92 0)
       (effects (font (size 1.27 1.27)) hide)
     )
@@
     (property "Reference" "U7" (id 0) (at 66.04 73.66 0))
     (property "Value" "XL4001" (id 1) (at 69.85 86.36 0))
-    (property "Footprint" "Package_SO:Texas_HTSOP-8-1EP_3.9x4.9mm_P1.27mm_EP2.95x4.9mm_Mask2.4x3.1mm_ThermalVias" (id 2) (at 69.85 83.82 0)
-      (effects (font (size 1.27 1.27)) hide)
-    )
+    (property "Footprint" "-local:Texas_HTSOP-8-1EP_3.9x4.9mm_P1.27mm_EP2.8x4.1mm_Mask2.8x4.1mm_ThermalVias" (id 2) (at 69.85 83.82 0)
+      (effects (font (size 1.27 1.27)) hide)
+    )

Commit message: using 10V zeners instead of 3V3 in all places. fixes #12, fixes #13
Parts:
- D24: value 3V3 -> 10V; LCSC Part Number C118713 -> C118715
Changed lines of the file:
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@@
       (effects (font (size 1.27 1.27)) (justify left))
     )
-    (property "Value" "3V3" (id 1) (at 101.6 45.72 90)
+    (property "Value" "10V" (id 1) (at 101.6 45.72 90)
       (effects (font (size 1.27 1.27)) (justify left))
     )
@@
       (effects (font (size 1.27 1.27)) hide)
     )
-    (property "Datasheet" "https://datasheet.lcsc.com/lcsc/1806121224_ST-Semtech-MM1Z5226B_C118713.pdf" (id 3) (at 101.6 43.18 0)
+    (property "Datasheet" "https://datasheet.lcsc.com/lcsc/1806070724_ST-Semtech-MM1Z5240B_C118715.pdf" (id 3) (at 101.6 43.18 0)
       (effects (font (size 1.27 1.27)) hide)
     )
-    (property "LCSC Part Number" "C118713" (id 4) (at 101.6 43.18 0)
+    (property "LCSC Part Number" "C118715" (id 4) (at 101.6 43.18 0)
       (effects (font (size 1.27 1.27)) hide)
     )

Commit message: fixing Q5 footprint and rerouting. fixes #1
Parts:
- Q5: symbol Device:Q_PMOS_GSD -> Device:Q_PMOS_GDS
Connections:
- net VIN: now also Q5.3 (S); no longer Q5.2 (S)
- net VIN_F: now also Q5.2 (D); no longer Q5.3 (D)
Changed lines of the file:
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@@
     (pin "1")
   )
-  (symbol (lib_id "Device:Q_PMOS_GSD") (at 96.52 40.64 90) (unit 1)
+  (symbol (lib_id "Device:Q_PMOS_GDS") (at 96.52 40.64 90) (unit 1)
     (in_bom yes) (on_board yes)
     (property "Reference" "Q5" (id 0) (at 96.52 31.75 90))
@@
       (effects (font (size 1.27 1.27)) hide)
     )
-    (property "Datasheet" "https://datasheet.lcsc.com/lcsc/2105241400_HUAYI-HYG210P06LQ1D_C2834760.pdf" (id 3) (at 96.52 40.64 0)
+    (property "Datasheet" "~" (id 3) (at 96.52 40.64 0)
       (effects (font (size 1.27 1.27)) hide)
     )
