File: maglock.kicad_sch (KiCad schematic)
At the start: 7 parts

Commit message: most stuff squeezed on board
Parts:
- LOGO2: footprint Symbol:OSHW-Logo2_7.3x6mm_SilkScreen -> Symbol:OSHW-Logo2_9.8x8mm_SilkScreen

Commit message: ERC, DRC and BOM fixes
Parts:
- H1, H2, H3, H4, H5, LOGO1, LOGO2: LCSC Part Number (none) -> -

Commit message: adding project info to sheet frames
Other:
- company: (none) -> makerspace.lt
- title: (none) -> MagLock
Changed lines of the file:
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@@
 (kicad_sch (version 20211123) (generator eeschema)
   (paper "A4")
+  (title_block
+    (title "MagLock")
+    (date "2022-07-20")
+    (rev "2.0")
+    (company "makerspace.lt")
+  )
   (junction (at 25.4 185.42) (diameter 0) (color 0 0 0 0)
   )
