File: maglock.kicad_sch (KiCad schematic)
At the start: 7 parts

Commit message: removing unreadable text from OSHW logo. fixes #15
Parts:
- LOGO2: footprint Symbol:OSHW-Logo2_9.8x8mm_SilkScreen -> Symbol:OSHW-Symbol_6.7x6mm_SilkScreen
Changed lines of the file:
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@@
       (effects (font (size 1.27 1.27)) hide)
     )
-    (property "Footprint" "Symbol:OSHW-Logo2_9.8x8mm_SilkScreen" (id 2) (at 55.88 182.88 0)
+    (property "Footprint" "Symbol:OSHW-Symbol_6.7x6mm_SilkScreen" (id 2) (at 55.88 182.88 0)
       (effects (font (size 1.27 1.27)) hide)
     )
@@
     )
     (path "/639f52c6-dbf2-4d74-80e1-6b05676c5315"
-      (reference "LOGO2") (unit 1) (value "Logo_Open_Hardware_Small") (footprint "Symbol:OSHW-Logo2_9.8x8mm_SilkScreen")
+      (reference "LOGO2") (unit 1) (value "Logo_Open_Hardware_Small") (footprint "Symbol:OSHW-Symbol_6.7x6mm_SilkScreen")
     )
     (path "/05705cd3-a12f-44ff-9d42-b34ea1caee0e/65cb4747-0618-4add-9fe4-125c843180ce"
