File: _main_soc.kicad_sch (KiCad schematic)
At the start: 15 parts, among them Q1 AO3400A, U4 DS18B20Z

Commit message: most stuff squeezed on board
Parts:
- removed C4: 1000u/10v, Capacitor_SMD:CP_Elec_10x10, symbol Device:C_Polarized
- added C4, C5, C6, C7, C8: 100u/10v, Capacitor_SMD:C_1206_3216Metric, symbol Device:C
- added J2: I2C0_128x32, -local:oled_i2c_128x32_ssd1306, symbol Connector:Conn_01x04_Female
- added J3: I2C1, Connector_PinSocket_2.54mm:PinSocket_1x04_P2.54mm_Vertical, symbol Connector:Conn_01x04_Female
- added J4: SPI1, Connector_PinSocket_2.54mm:PinSocket_1x06_P2.54mm_Vertical, symbol Connector:Conn_01x06_Female
- added J5: I2C0_128x64, -local:oled_i2c_128x64_ssd1306, symbol Connector:Conn_01x04_Female
Connections:
- net 3V3: now also C7.2, C8.2, J2.2 (Pin_2), J3.3 (Pin_3), J4.5 (Pin_5), J5.2 (Pin_2)
- net 5V: now also C4.2, C5.2, C6.2
- net GND: now also A1.MP (GND), C4.1, C5.1, C6.1, C7.1, C8.1, J2.1 (Pin_1), J3.4 (Pin_4), J4.6 (Pin_6), J5.1 (Pin_1)
- net REL1: now also A1.a12 (SIM_CLK/EINT/PA07)
- net REL2: now also A1.a10 (UART1_RX/PG07)
- net REL3: now also A1.a8 (UART1_TX/PG06)
- net _BUZZER: now also A1.a7 (PWM1/PA06); no longer A1.a12 (SIM_CLK/EINT/PA07)
- net I2C1_SDA: now reaches A1.a16 (I2C1_SDA/PA19)
- net I2C1_SDA: now also J3.1 (Pin_1)
- net I2C1_SCK: now reaches A1.a18 (I2C1_SCK/PA18)
- net I2C1_SCK: now also J3.2 (Pin_2)
- net SPI1_MOSI: now reaches A1.a19 (SPI1_MOSI/PA15)
- net SPI1_MOSI: now also J4.1 (Pin_1)
- net SPI1_MISO: now reaches A1.a21 (SPI1_MISO/PA16)
- net SPI1_MISO: now also J4.2 (Pin_2)
- net SPI1_CLK: now reaches A1.a23 (SPI1_CLK/PA14)
- net SPI1_CLK: now also J4.3 (Pin_3)
- net SPI1_CS: now reaches A1.a24 (SPI1_CS/PA13)
- net SPI1_CS: now also J4.4 (Pin_4)
- net I2C0_SDA: now reaches A1.a3 (I2C0_SDA/PA12)
- net I2C0_SDA: now also J2.4 (Pin_4), J5.4 (Pin_4)
- net I2C0_SCK: now reaches A1.a5 (I2C0_SCK/PA11)
- net I2C0_SCK: now also J2.3 (Pin_3), J5.3 (Pin_3)
- no-connect marks 10 -> 7
Other:
- moved on the sheet: D5, D6, R10, R11, R12

Commit message: general routing finished
Parts:
- removed C7: 100u/10v, Capacitor_SMD:C_1206_3216Metric, symbol Device:C
- added JP1: IO power selector, Jumper:SolderJumper-3_P1.3mm_Open_RoundedPad1.0x1.5mm, symbol Jumper:SolderJumper_3_Open
- added R13: 100, Resistor_SMD:R_0805_2012Metric, symbol Device:R
- added R6: 10K, Resistor_SMD:R_0805_2012Metric, symbol Device:R
- BZ1: footprint Buzzer_Beeper:Buzzer_12x9.5RM7.6 -> Buzzer_Beeper:MagneticBuzzer_CUI_CST-931RP-A; LCSC Part Number (none) -> C252935
- renumbered C8 to C7, D5 to D4, D6 to D5, D4 to D6, R12 to R10, R6 to R11, R7 to R12, R9 to R14, R10 to R7, R11 to R9
Connections:
- net 3V3: now also JP1.1 (A); no longer J2.2 (Pin_2), J3.3 (Pin_3), J4.5 (Pin_5), J5.2 (Pin_2)
- net 5V: now also J2.2 (Pin_2), J5.2 (Pin_2), JP1.3 (B)
- net GND: now also J3.1 (Pin_1), J4.1 (Pin_1); no longer J3.4 (Pin_4), J4.6 (Pin_6)
- net I2C1_SCK: now also J3.3 (Pin_3); no longer J3.2 (Pin_2)
- net I2C1_SDA: now also J3.4 (Pin_4); no longer J3.1 (Pin_1)
- net SPI1_CLK: now also J4.4 (Pin_4); no longer J4.3 (Pin_3)
- net SPI1_CS: now also J4.3 (Pin_3); no longer J4.4 (Pin_4)
- net SPI1_MISO: now also J4.5 (Pin_5); no longer J4.2 (Pin_2)
- net SPI1_MOSI: now also J4.6 (Pin_6); no longer J4.1 (Pin_1)
- net _BUZZER: now also R13.2; no longer Q1.1 (G), R8.1
- net at BZ1.2 (+), Q1.3 (D), R12.1: now also R6.2
- net at BZ1.1 (-), R11.1: now also R6.1
- new net: Q1.1 (G), R13.1, R8.1
- new net IOVCC: J3.2 (Pin_2), J4.2 (Pin_2), JP1.2 (C)
Other:
- note added: "Buzzer"
- note added: "Displays"
- note added: "GPIO Breakout"
- note added: "Power Indicators"
- note added: "Thermometer"
- moved on the sheet: BZ1, D4, D5, D6, J2, J3, J4, J5, Q1, R10, R11, R12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

Commit message: adding more info to silkscreen
Other:
- moved on the sheet: C7
Changed lines of the file:
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@@
 (kicad_sch (version 20211123) (generator eeschema)
   (paper "A4")
+  (junction (at 147.32 38.1) (diameter 0) (color 0 0 0 0)
+  )
   (junction (at 137.16 58.42) (diameter 0) (color 0 0 0 0)
   )
+  (junction (at 147.32 58.42) (diameter 0) (color 0 0 0 0)
+  )
   (junction (at 129.54 139.7) (diameter 0) (color 0 0 0 0)
   )
@@
   (junction (at 66.04 111.76) (diameter 0) (color 0 0 0 0)
   )
-  (junction (at 144.78 38.1) (diameter 0) (color 0 0 0 0)
-  )
   (junction (at 54.61 45.72) (diameter 0) (color 0 0 0 0)
   )
@@
   (junction (at 132.08 38.1) (diameter 0) (color 0 0 0 0)
   )
-  (junction (at 147.32 58.42) (diameter 0) (color 0 0 0 0)
-  )
   (junction (at 58.42 63.5) (diameter 0) (color 0 0 0 0)
   )
-  (junction (at 144.78 58.42) (diameter 0) (color 0 0 0 0)
-  )
   (junction (at 137.16 38.1) (diameter 0) (color 0 0 0 0)
   )
   (junction (at 132.08 58.42) (diameter 0) (color 0 0 0 0)
-  )
-  (junction (at 149.86 38.1) (diameter 0) (color 0 0 0 0)
   )
   (junction (at 54.61 38.1) (diameter 0) (color 0 0 0 0)
@@
     (stroke (width 0) (type default) (color 0 0 0 0))
   )
+  (wire (pts (xy 147.32 38.1) (xy 147.32 40.64))
+    (stroke (width 0) (type default) (color 0 0 0 0))
+  )
   (polyline (pts (xy 88.9 152.4) (xy 88.9 190.5))
     (stroke (width 0) (type default) (color 0 0 0 0))
   )
-  (wire (pts (xy 144.78 38.1) (xy 144.78 40.64))
-    (stroke (width 0) (type default) (color 0 0 0 0))
-  )
   (wire (pts (xy 223.52 101.6) (xy 228.6 101.6))
     (stroke (width 0) (type default) (color 0 0 0 0))
@@
     (stroke (width 0) (type default) (color 0 0 0 0))
   )
+  (wire (pts (xy 147.32 48.26) (xy 147.32 58.42))
+    (stroke (width 0) (type default) (color 0 0 0 0))
+  )
   (wire (pts (xy 147.32 139.7) (xy 152.4 139.7))
     (stroke (width 0) (type default) (color 0 0 0 0))
   )
-  (wire (pts (xy 149.86 38.1) (xy 158.75 38.1))
-    (stroke (width 0) (type default) (color 0 0 0 0))
-  )
   (wire (pts (xy 50.8 60.96) (xy 50.8 63.5))
     (stroke (width 0) (type default) (color 0 0 0 0))
   )
-  (wire (pts (xy 144.78 38.1) (xy 149.86 38.1))
-    (stroke (width 0) (type default) (color 0 0 0 0))
-  )
-  (wire (pts (xy 149.86 58.42) (xy 147.32 58.42))
+  (wire (pts (xy 147.32 38.1) (xy 158.75 38.1))
     (stroke (width 0) (type default) (color 0 0 0 0))
   )
@@
     (stroke (width 0) (type default) (color 0 0 0 0))
   )
-  (wire (pts (xy 149.86 48.26) (xy 149.86 58.42))
-    (stroke (width 0) (type default) (color 0 0 0 0))
-  )
-  (wire (pts (xy 144.78 48.26) (xy 144.78 58.42))
-    (stroke (width 0) (type default) (color 0 0 0 0))
-  )
   (wire (pts (xy 78.74 38.1) (xy 74.93 38.1))
     (stroke (width 0) (type default) (color 0 0 0 0))
@@
     (stroke (width 0) (type default) (color 0 0 0 0))
   )
-  (wire (pts (xy 149.86 38.1) (xy 149.86 40.64))
-    (stroke (width 0) (type default) (color 0 0 0 0))
-  )
   (wire (pts (xy 62.23 45.72) (xy 54.61 45.72))
     (stroke (width 0) (type default) (color 0 0 0 0))
@@
     (stroke (width 0) (type default) (color 0 0 0 0))
   )
-  (wire (pts (xy 137.16 38.1) (xy 144.78 38.1))
+  (wire (pts (xy 137.16 38.1) (xy 147.32 38.1))
     (stroke (width 0) (type default) (color 0 0 0 0))
   )
@@
     (effects (font (size 1.27 1.27)) (justify right))
   )
-  (hierarchical_label "3V3" (shape output) (at 149.86 57.15 0)
+  (hierarchical_label "3V3" (shape output) (at 147.32 57.15 0)
     (effects (font (size 1.27 1.27)) (justify left))
   )
@@
     (pin "1")
   )
-  (symbol (lib_id "Device:C") (at 149.86 44.45 0) (unit 1)
-    (in_bom yes) (on_board yes)
-    (property "Reference" "C7" (id 0) (at 148.59 43.18 90)
-      (effects (font (size 1.27 1.27)) (justify left))
-    )
-    (property "Value" "100u/10v" (id 1) (at 148.59 55.88 90)
-      (effects (font (size 1.27 1.27)) (justify left))
-    )
-    (property "Footprint" "Capacitor_SMD:C_1206_3216Metric" (id 2) (at 150.8252 48.26 0)
-      (effects (font (size 1.27 1.27)) hide)
-    )
-    (property "Datasheet" "https://datasheet.lcsc.com/lcsc/1811061115_Murata-Electronics-GRM31CR61A107ME05L_C312983.pdf" (id 3) (at 149.86 44.45 0)
-      (effects (font (size 1.27 1.27)) hide)
-    )
-    (property "LCSC Part Number" "C312983" (id 4) (at 149.86 44.45 0)
-      (effects (font (size 1.27 1.27)) hide)
-    )
-    (property "WE" "885012108012" (id 5) (at 149.86 44.45 0)
-      (effects (font (size 1.27 1.27)) hide)
-    )
+  (symbol (lib_id "Device:C") (at 147.32 44.45 0) (unit 1)
+    (in_bom yes) (on_board yes)
+    (property "Reference" "C7" (id 0) (at 146.05 43.18 90)
+      (effects (font (size 1.27 1.27)) (justify left))
+    )
+    (property "Value" "100u/10v" (id 1) (at 146.05 55.88 90)
+      (effects (font (size 1.27 1.27)) (justify left))
+    )
+    (property "Footprint" "Capacitor_SMD:C_1206_3216Metric" (id 2) (at 148.2852 48.26 0)
+      (effects (font (size 1.27 1.27)) hide)
+    )
+    (property "Datasheet" "https://datasheet.lcsc.com/lcsc/1811061115_Murata-Electronics-GRM31CR61A107ME05L_C312983.pdf" (id 3) (at 147.32 44.45 0)
+      (effects (font (size 1.27 1.27)) hide)
+    )
+    (property "LCSC Part Number" "C312983" (id 4) (at 147.32 44.45 0)
+      (effects (font (size 1.27 1.27)) hide)
+    )
+    (property "WE" "885012108012" (id 5) (at 147.32 44.45 0)
+      (effects (font (size 1.27 1.27)) hide)
+    )

Commit message: ERC, DRC and BOM fixes
Parts:
- A1, JP1: LCSC Part Number (none) -> -
- R11, R12, R13: value 100 -> 330
- R6, R8: value 10K -> 10k
Changed lines of the file:
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@@
+    (effects (font (size 1.27 1.27)) (justify left))
+  )
+  (hierarchical_label "3V3" (shape output) (at 165.1 177.8 0)
     (effects (font (size 1.27 1.27)) (justify left))
   )
@@
       (effects (font (size 1.27 1.27)) (justify left))
     )
-    (property "Value" "10K" (id 1) (at 58.42 60.96 90)
+    (property "Value" "10k" (id 1) (at 58.42 60.96 90)
       (effects (font (size 1.27 1.27)) (justify left))
     )
@@
       (effects (font (size 1.27 1.27)) (justify left))
     )
-    (property "Value" "100" (id 1) (at 67.31 55.88 90)
+    (property "Value" "330" (id 1) (at 67.31 55.88 90)
       (effects (font (size 1.27 1.27)) (justify left))
     )
@@
       (effects (font (size 1.27 1.27)) (justify left))
     )
-    (property "Value" "100" (id 1) (at 67.31 45.72 90)
+    (property "Value" "330" (id 1) (at 67.31 45.72 90)
       (effects (font (size 1.27 1.27)) (justify left))
     )
@@
     )
     (property "Datasheet" "~" (id 3) (at 220.98 55.88 0)
+      (effects (font (size 1.27 1.27)) hide)
+    )
+    (property "LCSC Part Number" "~" (id 4) (at 220.98 55.88 0)
       (effects (font (size 1.27 1.27)) hide)
     )
@@
     (pin "2")
   )
+  (symbol (lib_id "power:PWR_FLAG") (at 165.1 177.8 90) (unit 1)
+    (in_bom yes) (on_board yes) (fields_autoplaced)
+    (property "Reference" "#FLG08" (id 0) (at 163.195 177.8 0)
+      (effects (font (size 1.27 1.27)) hide)
+    )
+    (property "Value" "PWR_FLAG" (id 1) (at 160.02 177.8 0)
+      (effects (font (size 1.27 1.27)) hide)
+    )
+    (property "Footprint" "" (id 2) (at 165.1 177.8 0)
+      (effects (font (size 1.27 1.27)) hide)
+    )
+    (property "Datasheet" "~" (id 3) (at 165.1 177.8 0)
+      (effects (font (size 1.27 1.27)) hide)
+    )
+    (pin "1")
+  )
   (symbol (lib_id "Device:LED_Small_Filled") (at 72.39 45.72 0) (unit 1)
     (in_bom yes) (on_board yes)
@@
       (effects (font (size 1.27 1.27)) (justify left))
     )
-    (property "Value" "10K" (id 1) (at 54.61 43.18 90)
+    (property "Value" "10k" (id 1) (at 54.61 43.18 90)
       (effects (font (size 1.27 1.27)) (justify left))
     )
@@
       (effects (font (size 1.27 1.27)) hide)
     )
+    (property "LCSC Part Number" "~" (id 4) (at 246.38 55.88 0)
+      (effects (font (size 1.27 1.27)) hide)
+    )
     (pin "1")
     (pin "2")
@@
       (effects (font (size 1.27 1.27)) hide)
     )
+    (property "LCSC Part Number" "-" (id 4) (at 228.6 97.79 0)
+      (effects (font (size 1.27 1.27)) hide)
+    )
     (pin "1")
     (pin "2")
@@
       (effects (font (size 1.27 1.27)) (justify left))
     )
-    (property "Value" "100" (id 1) (at 67.31 38.1 90)
+    (property "Value" "330" (id 1) (at 67.31 38.1 90)
       (effects (font (size 1.27 1.27)) (justify left))
     )
@@
       (effects (font (size 1.27 1.27)) hide)
     )
+    (property "LCSC Part Number" "~" (id 4) (at 233.68 147.32 0)
+      (effects (font (size 1.27 1.27)) hide)
+    )
     (pin "1")
     (pin "2")
@@
       (effects (font (size 1.27 1.27)) hide)
     )
-    (property "LCSC Part Number" "~" (id 4) (at 137.16 99.06 0)
+    (property "LCSC Part Number" "-" (id 4) (at 137.16 99.06 0)
       (effects (font (size 1.27 1.27)) hide)
     )
@@
       (effects (font (size 1.27 1.27)) hide)
     )
+    (property "LCSC Part Number" "~" (id 4) (at 233.68 119.38 0)
+      (effects (font (size 1.27 1.27)) hide)
+    )

Commit message: adding project info to sheet frames
Other:
- company: (none) -> makerspace.lt
- title: (none) -> MagLock
Changed lines of the file:
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@@
 (kicad_sch (version 20211123) (generator eeschema)
   (paper "A4")
+  (title_block
+    (title "MagLock")
+    (date "2022-07-20")
+    (rev "2.0")
+    (company "makerspace.lt")
+  )
   (junction (at 147.32 38.1) (diameter 0) (color 0 0 0 0)
   )

Commit message: adding direction marker for buzzer. fixes #4
Parts:
- BZ1: footprint Buzzer_Beeper:MagneticBuzzer_CUI_CST-931RP-A -> -local:MagneticBuzzer_CUI_CST-931RP-A
Changed lines of the file:
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@@
     (property "Reference" "BZ1" (id 0) (at 46.99 38.1 0))
     (property "Value" "Buzzer" (id 1) (at 46.99 46.99 0))
-    (property "Footprint" "Buzzer_Beeper:MagneticBuzzer_CUI_CST-931RP-A" (id 2) (at 48.895 40.64 90)
+    (property "Footprint" "-local:MagneticBuzzer_CUI_CST-931RP-A" (id 2) (at 48.895 40.64 90)
       (effects (font (size 1.27 1.27)) hide)
     )

Commit message: adding OPI connectors to lcsc BOM. fixes 9
Parts:
- added XJaA1: Conn_02x13_Female_2.54, symbol Connector:Conn_01x01_Female
- added XJbA1: Conn_01x13_Female_2.54, symbol Connector:Conn_01x01_Female
- added XJcA1: Conn_01x03_Female_2.54, symbol Connector:Conn_01x01_Female
Connections:
- no-connect marks 7 -> 10
Other:
- note added: "OPI connectors for BOM"
Changed lines of the file:
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@@
   (no_connect (at 119.38 96.52))
   (no_connect (at 119.38 99.06))
+  (no_connect (at 110.49 179.07))
+  (no_connect (at 110.49 166.37))
+  (no_connect (at 110.49 172.72))
   (wire (pts (xy 50.8 40.64) (xy 50.8 38.1))
     (stroke (width 0) (type default) (color 0 0 0 0))
@@
     (stroke (width 0) (type default) (color 0 0 0 0))
   )
+  (polyline (pts (xy 101.6 190.5) (xy 160.02 190.5))
+    (stroke (width 0) (type default) (color 0 0 0 0))
+  )
   (wire (pts (xy 223.52 101.6) (xy 228.6 101.6))
     (stroke (width 0) (type default) (color 0 0 0 0))
@@
     (stroke (width 0) (type default) (color 0 0 0 0))
   )
+  (polyline (pts (xy 101.6 152.4) (xy 160.02 152.4))
+    (stroke (width 0) (type default) (color 0 0 0 0))
+  )
   (polyline (pts (xy 254 165.1) (xy 203.2 165.1))
     (stroke (width 0) (type default) (color 0 0 0 0))
@@
     (stroke (width 0) (type default) (color 0 0 0 0))
   )
+  (polyline (pts (xy 101.6 152.4) (xy 101.6 190.5))
+    (stroke (width 0) (type default) (color 0 0 0 0))
+  )
   (wire (pts (xy 78.74 38.1) (xy 74.93 38.1))
     (stroke (width 0) (type default) (color 0 0 0 0))
@@
   )
   (wire (pts (xy 139.7 139.7) (xy 142.24 139.7))
+    (stroke (width 0) (type default) (color 0 0 0 0))
+  )
+  (polyline (pts (xy 160.02 152.4) (xy 160.02 190.5))
     (stroke (width 0) (type default) (color 0 0 0 0))
   )
@@
     (effects (font (size 3 3) (thickness 0.6) bold) (justify left bottom))
   )
+  (text "OPI connectors for BOM" (at 102.87 158.75 0)
+    (effects (font (size 3 3) (thickness 0.6) bold) (justify left bottom))
+  )
   (text "Thermometer" (at 39.37 95.25 0)
     (effects (font (size 3 3) (thickness 0.6) bold) (justify left bottom))
@@
     (effects (font (size 1.27 1.27)) (justify left))
   )
-  (hierarchical_label "3V3" (shape output) (at 165.1 177.8 0)
+  (hierarchical_label "3V3" (shape output) (at 270.51 158.75 0)
     (effects (font (size 1.27 1.27)) (justify left))
   )
@@
     (pin "1")
   )
+  (symbol (lib_name "Conn_01x01_Female_1") (lib_id "Connector:Conn_01x01_Female") (at 115.57 166.37 0) (unit 1)
+    (in_bom yes) (on_board no) (fields_autoplaced)
+    (property "Reference" "XJaA1" (id 0) (at 116.84 165.0999 0)
+      (effects (font (size 1.27 1.27)) (justify left))
+    )
+    (property "Value" "Conn_02x13_Female_2.54" (id 1) (at 116.84 167.6399 0)
+      (effects (font (size 1.27 1.27)) (justify left))
+    )
+    (property "Footprint" "" (id 2) (at 115.57 166.37 0)
+      (effects (font (size 1.27 1.27)) hide)
+    )
+    (property "Datasheet" "~" (id 3) (at 115.57 166.37 0)
+      (effects (font (size 1.27 1.27)) hide)
+    )
+    (property "LCSC Part Number" "C350298" (id 4) (at 115.57 166.37 0)
+      (effects (font (size 1.27 1.27)) hide)
+    )
+    (pin "1")
+  )
   (symbol (lib_id "Device:R") (at 62.23 177.8 90) (unit 1)
     (in_bom yes) (on_board yes)
@@
     (pin "2")
   )
-  (symbol (lib_id "power:PWR_FLAG") (at 165.1 177.8 90) (unit 1)
+  (symbol (lib_id "Connector:Conn_01x01_Female") (at 115.57 179.07 0) (unit 1)
+    (in_bom yes) (on_board no) (fields_autoplaced)
+    (property "Reference" "XJcA1" (id 0) (at 116.84 177.7999 0)
+      (effects (font (size 1.27 1.27)) (justify left))
+    )
+    (property "Value" "Conn_01x03_Female_2.54" (id 1) (at 116.84 180.3399 0)
+      (effects (font (size 1.27 1.27)) (justify left))
+    )
+    (property "Footprint" "" (id 2) (at 115.57 179.07 0)
+      (effects (font (size 1.27 1.27)) hide)
+    )
+    (property "Datasheet" "~" (id 3) (at 115.57 179.07 0)
+      (effects (font (size 1.27 1.27)) hide)
+    )
+    (property "LCSC Part Number" "C2935974" (id 4) (at 115.57 179.07 0)
+      (effects (font (size 1.27 1.27)) hide)
+    )
+    (pin "1")
+  )
+  (symbol (lib_id "power:PWR_FLAG") (at 270.51 158.75 90) (unit 1)
     (in_bom yes) (on_board yes) (fields_autoplaced)
-    (property "Reference" "#FLG08" (id 0) (at 163.195 177.8 0)
-      (effects (font (size 1.27 1.27)) hide)
-    )
-    (property "Value" "PWR_FLAG" (id 1) (at 160.02 177.8 0)
-      (effects (font (size 1.27 1.27)) hide)
-    )
-    (property "Footprint" "" (id 2) (at 165.1 177.8 0)
-      (effects (font (size 1.27 1.27)) hide)
-    )
-    (property "Datasheet" "~" (id 3) (at 165.1 177.8 0)
+    (property "Reference" "#FLG08" (id 0) (at 268.605 158.75 0)
+      (effects (font (size 1.27 1.27)) hide)
+    )
+    (property "Value" "PWR_FLAG" (id 1) (at 265.43 158.75 0)
+      (effects (font (size 1.27 1.27)) hide)
+    )
+    (property "Footprint" "" (id 2) (at 270.51 158.75 0)
+      (effects (font (size 1.27 1.27)) hide)
+    )
+    (property "Datasheet" "~" (id 3) (at 270.51 158.75 0)
       (effects (font (size 1.27 1.27)) hide)
     )
@@
     (pin "2")
   )
+  (symbol (lib_name "Conn_01x01_Female_2") (lib_id "Connector:Conn_01x01_Female") (at 115.57 172.72 0) (unit 1)
+    (in_bom yes) (on_board no) (fields_autoplaced)
+    (property "Reference" "XJbA1" (id 0) (at 116.84 171.4499 0)
+      (effects (font (size 1.27 1.27)) (justify left))
+    )
+    (property "Value" "Conn_01x13_Female_2.54" (id 1) (at 116.84 173.9899 0)
+      (effects (font (size 1.27 1.27)) (justify left))
+    )
+    (property "Footprint" "" (id 2) (at 115.57 172.72 0)
+      (effects (font (size 1.27 1.27)) hide)
+    )
+    (property "Datasheet" "~" (id 3) (at 115.57 172.72 0)
+      (effects (font (size 1.27 1.27)) hide)
+    )
+    (property "LCSC Part Number" "C52709" (id 4) (at 115.57 172.72 0)
+      (effects (font (size 1.27 1.27)) hide)
+    )
+    (pin "1")
+  )
   (symbol (lib_id "Connector:Conn_01x04_Female") (at 246.38 55.88 0) (mirror x) (unit 1)
