File: _main_soc.kicad_sch (KiCad schematic)
At the start: 28 parts, among them J2 I2C0_128x32, J3 I2C1, J4 SPI1, J5 I2C0_128x64, Q1 AO3400A, U4 DS18B20Z

Commit message: making buzzer louder by using 0R in place of current limiter. fixes #10
Parts:
- R11: value 330 -> 0
Changed lines of the file:
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@@
   (no_connect (at 119.38 96.52))
   (no_connect (at 119.38 99.06))
+  (no_connect (at 110.49 172.72))
   (no_connect (at 110.49 179.07))
   (no_connect (at 110.49 166.37))
-  (no_connect (at 110.49 172.72))
   (wire (pts (xy 50.8 40.64) (xy 50.8 38.1))
     (stroke (width 0) (type default) (color 0 0 0 0))
@@
       (effects (font (size 1.27 1.27)) (justify left))
     )
-    (property "Value" "330" (id 1) (at 67.31 38.1 90)
-      (effects (font (size 1.27 1.27)) (justify left))
-    )
+    (property "Value" "0" (id 1) (at 67.31 38.1 90)
+      (effects (font (size 1.27 1.27)) (justify left))
+    )

Commit message: removing an unnecessary resistor from OPI 5V indicator. fixes #6
Parts:
- removed R9: 1k, Resistor_SMD:R_0805_2012Metric, symbol Device:R
- R7: value 1k -> 4k7
Connections:
- net at D4.1 (K): now also R7.2
Other:
- moved on the sheet: R7
Changed lines of the file:
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@@
   (junction (at 147.32 139.7) (diameter 0) (color 0 0 0 0)
   )
+  (junction (at 132.08 139.7) (diameter 0) (color 0 0 0 0)
+  )
+  (junction (at 50.8 45.72) (diameter 0) (color 0 0 0 0)
+  )
+  (junction (at 139.7 139.7) (diameter 0) (color 0 0 0 0)
+  )
+  (junction (at 74.93 38.1) (diameter 0) (color 0 0 0 0)
+  )
+  (junction (at 66.04 111.76) (diameter 0) (color 0 0 0 0)
+  )
+  (junction (at 54.61 45.72) (diameter 0) (color 0 0 0 0)
+  )
+  (junction (at 137.16 139.7) (diameter 0) (color 0 0 0 0)
+  )
+  (junction (at 142.24 139.7) (diameter 0) (color 0 0 0 0)
+  )
+  (junction (at 129.54 58.42) (diameter 0) (color 0 0 0 0)
+  )
+  (junction (at 134.62 139.7) (diameter 0) (color 0 0 0 0)
+  )
+  (junction (at 58.42 55.88) (diameter 0) (color 0 0 0 0)
+  )
+  (junction (at 132.08 38.1) (diameter 0) (color 0 0 0 0)
+  )
+  (junction (at 58.42 63.5) (diameter 0) (color 0 0 0 0)
+  )
+  (junction (at 137.16 38.1) (diameter 0) (color 0 0 0 0)
+  )
+  (junction (at 132.08 58.42) (diameter 0) (color 0 0 0 0)
+  )
+  (junction (at 54.61 38.1) (diameter 0) (color 0 0 0 0)
+  )
+  (junction (at 66.04 119.38) (diameter 0) (color 0 0 0 0)
+  )
   (junction (at 50.8 177.8) (diameter 0) (color 0 0 0 0)
-  )
-  (junction (at 132.08 139.7) (diameter 0) (color 0 0 0 0)
-  )
-  (junction (at 50.8 45.72) (diameter 0) (color 0 0 0 0)
-  )
-  (junction (at 139.7 139.7) (diameter 0) (color 0 0 0 0)
-  )
-  (junction (at 74.93 38.1) (diameter 0) (color 0 0 0 0)
-  )
-  (junction (at 66.04 111.76) (diameter 0) (color 0 0 0 0)
-  )
-  (junction (at 54.61 45.72) (diameter 0) (color 0 0 0 0)
-  )
-  (junction (at 137.16 139.7) (diameter 0) (color 0 0 0 0)
-  )
-  (junction (at 142.24 139.7) (diameter 0) (color 0 0 0 0)
-  )
-  (junction (at 129.54 58.42) (diameter 0) (color 0 0 0 0)
-  )
-  (junction (at 134.62 139.7) (diameter 0) (color 0 0 0 0)
-  )
-  (junction (at 58.42 55.88) (diameter 0) (color 0 0 0 0)
-  )
-  (junction (at 132.08 38.1) (diameter 0) (color 0 0 0 0)
-  )
-  (junction (at 58.42 63.5) (diameter 0) (color 0 0 0 0)
-  )
-  (junction (at 137.16 38.1) (diameter 0) (color 0 0 0 0)
-  )
-  (junction (at 132.08 58.42) (diameter 0) (color 0 0 0 0)
-  )
-  (junction (at 54.61 38.1) (diameter 0) (color 0 0 0 0)
-  )
-  (junction (at 66.04 119.38) (diameter 0) (color 0 0 0 0)
   )
   (no_connect (at 119.38 119.38))
@@
   (no_connect (at 119.38 96.52))
   (no_connect (at 119.38 99.06))
-  (no_connect (at 110.49 166.37))
   (no_connect (at 110.49 179.07))
   (no_connect (at 110.49 172.72))
+  (no_connect (at 110.49 166.37))
   (wire (pts (xy 50.8 40.64) (xy 50.8 38.1))
     (stroke (width 0) (type default) (color 0 0 0 0))
@@
     (stroke (width 0) (type default) (color 0 0 0 0))
   )
+  (wire (pts (xy 58.42 165.1) (xy 50.8 165.1))
+    (stroke (width 0) (type default) (color 0 0 0 0))
+  )
   (polyline (pts (xy 38.1 90.17) (xy 38.1 139.7))
     (stroke (width 0) (type default) (color 0 0 0 0))
@@
     (stroke (width 0) (type default) (color 0 0 0 0))
   )
+  (polyline (pts (xy 38.1 25.4) (xy 38.1 76.2))
+    (stroke (width 0) (type default) (color 0 0 0 0))
+  )
   (wire (pts (xy 50.8 165.1) (xy 50.8 177.8))
-    (stroke (width 0) (type default) (color 0 0 0 0))
-  )
-  (polyline (pts (xy 38.1 25.4) (xy 38.1 76.2))
     (stroke (width 0) (type default) (color 0 0 0 0))
   )
@@
     (pin "1")
   )
-  (symbol (lib_id "Device:R") (at 62.23 165.1 90) (unit 1)
-    (in_bom yes) (on_board yes)
-    (property "Reference" "R9" (id 0) (at 63.5 162.56 90)
-      (effects (font (size 1.27 1.27)) (justify left))
-    )
-    (property "Value" "1k" (id 1) (at 63.5 165.1 90)
-      (effects (font (size 1.27 1.27)) (justify left))
-    )
-    (property "Footprint" "Resistor_SMD:R_0805_2012Metric" (id 2) (at 62.23 166.878 90)
-      (effects (font (size 1.27 1.27)) hide)
-    )
-    (property "Datasheet" "~" (id 3) (at 62.23 165.1 0)
-      (effects (font (size 1.27 1.27)) hide)
-    )
-    (property "LCSC Part Number" "~" (id 4) (at 62.23 165.1 0)
-      (effects (font (size 1.27 1.27)) hide)
-    )
-    (pin "1")
-    (pin "2")
-  )
   (symbol (lib_id "Transistor_FET:AO3400A") (at 53.34 55.88 0) (mirror y) (unit 1)
     (in_bom yes) (on_board yes)
@@
     (pin "1")
   )
-  (symbol (lib_id "Device:R") (at 54.61 165.1 90) (unit 1)
-    (in_bom yes) (on_board yes)
-    (property "Reference" "R7" (id 0) (at 55.88 162.56 90)
-      (effects (font (size 1.27 1.27)) (justify left))
-    )
-    (property "Value" "1k" (id 1) (at 55.88 165.1 90)
-      (effects (font (size 1.27 1.27)) (justify left))
-    )
-    (property "Footprint" "Resistor_SMD:R_0805_2012Metric" (id 2) (at 54.61 166.878 90)
-      (effects (font (size 1.27 1.27)) hide)
-    )
-    (property "Datasheet" "~" (id 3) (at 54.61 165.1 0)
-      (effects (font (size 1.27 1.27)) hide)
-    )
-    (property "LCSC Part Number" "~" (id 4) (at 54.61 165.1 0)
-      (effects (font (size 1.27 1.27)) hide)
-    )
+  (symbol (lib_id "Device:R") (at 62.23 165.1 90) (unit 1)
+    (in_bom yes) (on_board yes)
+    (property "Reference" "R7" (id 0) (at 63.5 162.56 90)
+      (effects (font (size 1.27 1.27)) (justify left))
+    )
+    (property "Value" "4k7" (id 1) (at 63.5 165.1 90)
+      (effects (font (size 1.27 1.27)) (justify left))
+    )
+    (property "Footprint" "Resistor_SMD:R_0805_2012Metric" (id 2) (at 62.23 166.878 90)
+      (effects (font (size 1.27 1.27)) hide)
+    )
+    (property "Datasheet" "~" (id 3) (at 62.23 165.1 0)
+      (effects (font (size 1.27 1.27)) hide)
+    )
+    (property "LCSC Part Number" "~" (id 4) (at 62.23 165.1 0)
+      (effects (font (size 1.27 1.27)) hide)
+    )
