File: _inputs.kicad_sch (KiCad schematic)
At the start: 32 parts, among them SW1 2pin, SW2 2pin, SW3 2pin, SW4 2pin

Commit message: most stuff squeezed on board
Parts:
- renumbered C6 to C10, C7 to C11, C8 to C12, C5 to C9
Changed lines of the file:
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@@
   (symbol (lib_id "power:GND") (at 156.21 86.36 0) (unit 1)
     (in_bom yes) (on_board yes)
-    (property "Reference" "#PWR015" (id 0) (at 156.21 92.71 0)
+    (property "Reference" "#PWR019" (id 0) (at 156.21 92.71 0)
       (effects (font (size 1.27 1.27)) hide)
     )
@@
   (symbol (lib_id "power:GND") (at 156.21 111.76 0) (unit 1)
     (in_bom yes) (on_board yes)
-    (property "Reference" "#PWR016" (id 0) (at 156.21 118.11 0)
+    (property "Reference" "#PWR020" (id 0) (at 156.21 118.11 0)
       (effects (font (size 1.27 1.27)) hide)
     )
@@
   )
   (symbol (lib_id "Connector:Conn_01x02_Male") (at 93.98 57.15 180) (unit 1)
-    (in_bom yes) (on_board yes) (fields_autoplaced)
+    (in_bom yes) (on_board no) (fields_autoplaced)
     (property "Reference" "XSW1" (id 0) (at 94.615 49.53 0))
     (property "Value" "2pin" (id 1) (at 94.615 52.07 0))
@@
   (symbol (lib_id "power:GND") (at 156.21 60.96 0) (unit 1)
     (in_bom yes) (on_board yes)
-    (property "Reference" "#PWR014" (id 0) (at 156.21 67.31 0)
+    (property "Reference" "#PWR018" (id 0) (at 156.21 67.31 0)
       (effects (font (size 1.27 1.27)) hide)
     )
@@
   (symbol (lib_id "Device:C") (at 149.86 57.15 0) (unit 1)
     (in_bom yes) (on_board yes)
-    (property "Reference" "C5" (id 0) (at 149.86 54.61 0)
+    (property "Reference" "C9" (id 0) (at 149.86 54.61 0)
       (effects (font (size 1.27 1.27)) (justify left))
     )
@@
   )
   (symbol (lib_id "Connector:Conn_01x02_Male") (at 93.98 107.95 180) (unit 1)
-    (in_bom yes) (on_board yes) (fields_autoplaced)
+    (in_bom yes) (on_board no) (fields_autoplaced)
     (property "Reference" "XSW3" (id 0) (at 94.615 100.33 0))
     (property "Value" "2pin" (id 1) (at 94.615 102.87 0))
@@
   (symbol (lib_id "power:GND") (at 156.21 137.16 0) (unit 1)
     (in_bom yes) (on_board yes)
-    (property "Reference" "#PWR017" (id 0) (at 156.21 143.51 0)
+    (property "Reference" "#PWR021" (id 0) (at 156.21 143.51 0)
       (effects (font (size 1.27 1.27)) hide)
     )
@@
   (symbol (lib_id "Device:C") (at 149.86 82.55 0) (unit 1)
     (in_bom yes) (on_board yes)
-    (property "Reference" "C6" (id 0) (at 149.86 80.01 0)
+    (property "Reference" "C10" (id 0) (at 149.86 80.01 0)
       (effects (font (size 1.27 1.27)) (justify left))
     )
@@
   (symbol (lib_id "Device:C") (at 149.86 107.95 0) (unit 1)
     (in_bom yes) (on_board yes)
-    (property "Reference" "C7" (id 0) (at 149.86 105.41 0)
+    (property "Reference" "C11" (id 0) (at 149.86 105.41 0)
       (effects (font (size 1.27 1.27)) (justify left))
     )
@@
   (symbol (lib_id "Device:C") (at 149.86 133.35 0) (unit 1)
     (in_bom yes) (on_board yes)
-    (property "Reference" "C8" (id 0) (at 149.86 130.81 0)
+    (property "Reference" "C12" (id 0) (at 149.86 130.81 0)
       (effects (font (size 1.27 1.27)) (justify left))
     )
@@
   )
   (symbol (lib_id "Connector:Conn_01x02_Male") (at 93.98 82.55 180) (unit 1)
-    (in_bom yes) (on_board yes) (fields_autoplaced)
+    (in_bom yes) (on_board no) (fields_autoplaced)
     (property "Reference" "XSW2" (id 0) (at 94.615 74.93 0))
     (property "Value" "2pin" (id 1) (at 94.615 77.47 0))
@@
   )
   (symbol (lib_id "Connector:Conn_01x02_Male") (at 93.98 133.35 180) (unit 1)
-    (in_bom yes) (on_board yes) (fields_autoplaced)
+    (in_bom yes) (on_board no) (fields_autoplaced)
     (property "Reference" "XSW4" (id 0) (at 94.615 125.73 0))
     (property "Value" "2pin" (id 1) (at 94.615 128.27 0))

Commit message: general routing finished
Parts:
- renumbered R13 to R15, R14 to R16, R15 to R17, R16 to R18, R17 to R19, R18 to R20, R19 to R21, R20 to R22, R21 to R23, R22 to R24, R23 to R25, R24 to R26, R25 to R27, R26 to R28, R27 to R29, R28 to R30
Changed lines of the file:
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@@
   (symbol (lib_id "Device:R") (at 162.56 78.74 90) (unit 1)
     (in_bom yes) (on_board yes)
-    (property "Reference" "R24" (id 0) (at 163.83 81.28 90)
+    (property "Reference" "R26" (id 0) (at 163.83 81.28 90)
       (effects (font (size 1.27 1.27)) (justify left))
     )
@@
   (symbol (lib_id "power:GND") (at 156.21 86.36 0) (unit 1)
     (in_bom yes) (on_board yes)
-    (property "Reference" "#PWR019" (id 0) (at 156.21 92.71 0)
+    (property "Reference" "#PWR020" (id 0) (at 156.21 92.71 0)
       (effects (font (size 1.27 1.27)) hide)
     )
@@
   (symbol (lib_id "Device:R") (at 143.51 86.36 90) (unit 1)
     (in_bom yes) (on_board yes)
-    (property "Reference" "R16" (id 0) (at 143.51 83.82 90)
+    (property "Reference" "R18" (id 0) (at 143.51 83.82 90)
       (effects (font (size 1.27 1.27)) (justify left))
     )
@@
   (symbol (lib_id "power:GND") (at 156.21 111.76 0) (unit 1)
     (in_bom yes) (on_board yes)
-    (property "Reference" "#PWR020" (id 0) (at 156.21 118.11 0)
+    (property "Reference" "#PWR021" (id 0) (at 156.21 118.11 0)
       (effects (font (size 1.27 1.27)) hide)
     )
@@
   (symbol (lib_id "power:GND") (at 156.21 60.96 0) (unit 1)
     (in_bom yes) (on_board yes)
-    (property "Reference" "#PWR018" (id 0) (at 156.21 67.31 0)
+    (property "Reference" "#PWR019" (id 0) (at 156.21 67.31 0)
       (effects (font (size 1.27 1.27)) hide)
     )
@@
   (symbol (lib_id "Device:R") (at 162.56 50.8 90) (unit 1)
     (in_bom yes) (on_board yes)
-    (property "Reference" "R21" (id 0) (at 163.83 48.26 90)
+    (property "Reference" "R23" (id 0) (at 163.83 48.26 90)
       (effects (font (size 1.27 1.27)) (justify left))
     )
@@
   (symbol (lib_id "Device:R") (at 162.56 101.6 90) (unit 1)
     (in_bom yes) (on_board yes)
-    (property "Reference" "R25" (id 0) (at 163.83 99.06 90)
+    (property "Reference" "R27" (id 0) (at 163.83 99.06 90)
       (effects (font (size 1.27 1.27)) (justify left))
     )
@@
   (symbol (lib_id "Device:R") (at 143.51 137.16 90) (unit 1)
     (in_bom yes) (on_board yes)
-    (property "Reference" "R20" (id 0) (at 143.51 134.62 90)
+    (property "Reference" "R22" (id 0) (at 143.51 134.62 90)
       (effects (font (size 1.27 1.27)) (justify left))
     )
@@
   (symbol (lib_id "Device:R") (at 162.56 127 90) (unit 1)
     (in_bom yes) (on_board yes)
-    (property "Reference" "R27" (id 0) (at 163.83 124.46 90)
+    (property "Reference" "R29" (id 0) (at 163.83 124.46 90)
       (effects (font (size 1.27 1.27)) (justify left))
     )
@@
   (symbol (lib_id "Device:R") (at 143.51 60.96 90) (unit 1)
     (in_bom yes) (on_board yes)
-    (property "Reference" "R14" (id 0) (at 143.51 58.42 90)
+    (property "Reference" "R16" (id 0) (at 143.51 58.42 90)
       (effects (font (size 1.27 1.27)) (justify left))
     )
@@
   (symbol (lib_id "Device:R") (at 143.51 101.6 90) (unit 1)
     (in_bom yes) (on_board yes)
-    (property "Reference" "R17" (id 0) (at 143.51 99.06 90)
+    (property "Reference" "R19" (id 0) (at 143.51 99.06 90)
       (effects (font (size 1.27 1.27)) (justify left))
     )
@@
   (symbol (lib_id "Device:R") (at 143.51 127 90) (unit 1)
     (in_bom yes) (on_board yes)
-    (property "Reference" "R19" (id 0) (at 143.51 124.46 90)
+    (property "Reference" "R21" (id 0) (at 143.51 124.46 90)
       (effects (font (size 1.27 1.27)) (justify left))
     )
@@
   (symbol (lib_id "Device:R") (at 162.56 76.2 90) (unit 1)
     (in_bom yes) (on_board yes)
-    (property "Reference" "R23" (id 0) (at 163.83 73.66 90)
+    (property "Reference" "R25" (id 0) (at 163.83 73.66 90)
       (effects (font (size 1.27 1.27)) (justify left))
     )
@@
   (symbol (lib_id "power:GND") (at 156.21 137.16 0) (unit 1)
     (in_bom yes) (on_board yes)
-    (property "Reference" "#PWR021" (id 0) (at 156.21 143.51 0)
+    (property "Reference" "#PWR022" (id 0) (at 156.21 143.51 0)
       (effects (font (size 1.27 1.27)) hide)
     )
@@
   (symbol (lib_id "Device:R") (at 162.56 104.14 90) (unit 1)
     (in_bom yes) (on_board yes)
-    (property "Reference" "R26" (id 0) (at 163.83 106.68 90)
+    (property "Reference" "R28" (id 0) (at 163.83 106.68 90)
       (effects (font (size 1.27 1.27)) (justify left))
     )
@@
   (symbol (lib_id "Device:R") (at 143.51 111.76 90) (unit 1)
     (in_bom yes) (on_board yes)
-    (property "Reference" "R18" (id 0) (at 143.51 109.22 90)
+    (property "Reference" "R20" (id 0) (at 143.51 109.22 90)
       (effects (font (size 1.27 1.27)) (justify left))
     )
@@
   (symbol (lib_id "Device:R") (at 143.51 50.8 90) (unit 1)
     (in_bom yes) (on_board yes)
-    (property "Reference" "R13" (id 0) (at 143.51 48.26 90)
+    (property "Reference" "R15" (id 0) (at 143.51 48.26 90)
       (effects (font (size 1.27 1.27)) (justify left))
     )
@@
   (symbol (lib_id "Device:R") (at 143.51 76.2 90) (unit 1)
     (in_bom yes) (on_board yes)
-    (property "Reference" "R15" (id 0) (at 143.51 73.66 90)
+    (property "Reference" "R17" (id 0) (at 143.51 73.66 90)
       (effects (font (size 1.27 1.27)) (justify left))
     )
@@
   (symbol (lib_id "Device:R") (at 162.56 129.54 90) (unit 1)
     (in_bom yes) (on_board yes)
-    (property "Reference" "R28" (id 0) (at 163.83 132.08 90)
+    (property "Reference" "R30" (id 0) (at 163.83 132.08 90)
       (effects (font (size 1.27 1.27)) (justify left))
     )
@@
   (symbol (lib_id "Device:R") (at 162.56 53.34 90) (unit 1)
     (in_bom yes) (on_board yes)
-    (property "Reference" "R22" (id 0) (at 163.83 55.88 90)
-      (effects (font (size 1.27 1.27)) (justify left))
-    )
+    (property "Reference" "R24" (id 0) (at 163.83 55.88 90)
+      (effects (font (size 1.27 1.27)) (justify left))
+    )

Commit message: adding documentation layers
Other:
- moved on the sheet: XSW1, XSW2, XSW3, XSW4
Changed lines of the file:
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@@
   )
   (symbol (lib_id "Connector:Conn_01x02_Female") (at 133.35 107.95 180) (unit 1)
-    (in_bom yes) (on_board yes) (fields_autoplaced)
-    (property "Reference" "SW3" (id 0) (at 133.985 100.33 0))
-    (property "Value" "2pin" (id 1) (at 133.985 102.87 0))
+    (in_bom yes) (on_board yes)
+    (property "Reference" "SW3" (id 0) (at 135.89 100.33 0))
+    (property "Value" "2pin" (id 1) (at 135.89 102.87 0))
     (property "Footprint" "TerminalBlock_Phoenix:TerminalBlock_Phoenix_PT-1,5-2-3.5-H_1x02_P3.50mm_Horizontal" (id 2) (at 133.35 107.95 0)
       (effects (font (size 1.27 1.27)) hide)
@@
   )
   (symbol (lib_id "Connector:Conn_01x02_Female") (at 133.35 57.15 180) (unit 1)
-    (in_bom yes) (on_board yes) (fields_autoplaced)
-    (property "Reference" "SW1" (id 0) (at 133.985 49.53 0))
-    (property "Value" "2pin" (id 1) (at 133.985 52.07 0))
+    (in_bom yes) (on_board yes)
+    (property "Reference" "SW1" (id 0) (at 135.89 49.53 0))
+    (property "Value" "2pin" (id 1) (at 135.89 52.07 0))
     (property "Footprint" "TerminalBlock_Phoenix:TerminalBlock_Phoenix_PT-1,5-2-3.5-H_1x02_P3.50mm_Horizontal" (id 2) (at 133.35 57.15 0)
       (effects (font (size 1.27 1.27)) hide)
@@
     (pin "1")
   )
-  (symbol (lib_id "Connector:Conn_01x02_Male") (at 93.98 57.15 180) (unit 1)
-    (in_bom yes) (on_board no) (fields_autoplaced)
-    (property "Reference" "XSW1" (id 0) (at 94.615 49.53 0))
-    (property "Value" "2pin" (id 1) (at 94.615 52.07 0))
-    (property "Footprint" "" (id 2) (at 93.98 57.15 0)
-      (effects (font (size 1.27 1.27)) hide)
-    )
-    (property "Datasheet" "https://datasheet.lcsc.com/lcsc/1912111437_JILN-JL15EDGK-35002G01_C393013.pdf" (id 3) (at 93.98 57.15 0)
-      (effects (font (size 1.27 1.27)) hide)
-    )
-    (property "LCSC Part Number" "C393013" (id 4) (at 93.98 57.15 0)
+  (symbol (lib_id "Connector:Conn_01x02_Male") (at 133.35 57.15 180) (unit 1)
+    (in_bom yes) (on_board no)
+    (property "Reference" "XSW1" (id 0) (at 128.27 49.53 0))
+    (property "Value" "2pin" (id 1) (at 128.27 52.07 0))
+    (property "Footprint" "" (id 2) (at 133.35 57.15 0)
+      (effects (font (size 1.27 1.27)) hide)
+    )
+    (property "Datasheet" "https://datasheet.lcsc.com/lcsc/1912111437_JILN-JL15EDGK-35002G01_C393013.pdf" (id 3) (at 133.35 57.15 0)
+      (effects (font (size 1.27 1.27)) hide)
+    )
+    (property "LCSC Part Number" "C393013" (id 4) (at 133.35 57.15 0)
       (effects (font (size 1.27 1.27)) hide)
     )
@@
     (pin "2")
   )
-  (symbol (lib_id "Connector:Conn_01x02_Male") (at 93.98 107.95 180) (unit 1)
-    (in_bom yes) (on_board no) (fields_autoplaced)
-    (property "Reference" "XSW3" (id 0) (at 94.615 100.33 0))
-    (property "Value" "2pin" (id 1) (at 94.615 102.87 0))
-    (property "Footprint" "" (id 2) (at 93.98 107.95 0)
-      (effects (font (size 1.27 1.27)) hide)
-    )
-    (property "Datasheet" "https://datasheet.lcsc.com/lcsc/1912111437_JILN-JL15EDGK-35002G01_C393013.pdf" (id 3) (at 93.98 107.95 0)
-      (effects (font (size 1.27 1.27)) hide)
-    )
-    (property "LCSC Part Number" "C393013" (id 4) (at 93.98 107.95 0)
+  (symbol (lib_id "Connector:Conn_01x02_Male") (at 133.35 107.95 180) (unit 1)
+    (in_bom yes) (on_board no)
+    (property "Reference" "XSW3" (id 0) (at 128.27 100.33 0))
+    (property "Value" "2pin" (id 1) (at 128.27 102.87 0))
+    (property "Footprint" "" (id 2) (at 133.35 107.95 0)
+      (effects (font (size 1.27 1.27)) hide)
+    )
+    (property "Datasheet" "https://datasheet.lcsc.com/lcsc/1912111437_JILN-JL15EDGK-35002G01_C393013.pdf" (id 3) (at 133.35 107.95 0)
+      (effects (font (size 1.27 1.27)) hide)
+    )
+    (property "LCSC Part Number" "C393013" (id 4) (at 133.35 107.95 0)
       (effects (font (size 1.27 1.27)) hide)
     )
@@
     (pin "2")
   )
-  (symbol (lib_id "Connector:Conn_01x02_Male") (at 93.98 82.55 180) (unit 1)
-    (in_bom yes) (on_board no) (fields_autoplaced)
-    (property "Reference" "XSW2" (id 0) (at 94.615 74.93 0))
-    (property "Value" "2pin" (id 1) (at 94.615 77.47 0))
-    (property "Footprint" "" (id 2) (at 93.98 82.55 0)
-      (effects (font (size 1.27 1.27)) hide)
-    )
-    (property "Datasheet" "https://datasheet.lcsc.com/lcsc/1912111437_JILN-JL15EDGK-35002G01_C393013.pdf" (id 3) (at 93.98 82.55 0)
-      (effects (font (size 1.27 1.27)) hide)
-    )
-    (property "LCSC Part Number" "C393013" (id 4) (at 93.98 82.55 0)
+  (symbol (lib_id "Connector:Conn_01x02_Male") (at 133.35 82.55 180) (unit 1)
+    (in_bom yes) (on_board no)
+    (property "Reference" "XSW2" (id 0) (at 128.27 74.93 0))
+    (property "Value" "2pin" (id 1) (at 128.27 77.47 0))
+    (property "Footprint" "" (id 2) (at 133.35 82.55 0)
+      (effects (font (size 1.27 1.27)) hide)
+    )
+    (property "Datasheet" "https://datasheet.lcsc.com/lcsc/1912111437_JILN-JL15EDGK-35002G01_C393013.pdf" (id 3) (at 133.35 82.55 0)
+      (effects (font (size 1.27 1.27)) hide)
+    )
+    (property "LCSC Part Number" "C393013" (id 4) (at 133.35 82.55 0)
       (effects (font (size 1.27 1.27)) hide)
     )
@@
     (pin "2")
   )
-  (symbol (lib_id "Connector:Conn_01x02_Male") (at 93.98 133.35 180) (unit 1)
-    (in_bom yes) (on_board no) (fields_autoplaced)
-    (property "Reference" "XSW4" (id 0) (at 94.615 125.73 0))
-    (property "Value" "2pin" (id 1) (at 94.615 128.27 0))
-    (property "Footprint" "" (id 2) (at 93.98 133.35 0)
-      (effects (font (size 1.27 1.27)) hide)
-    )
-    (property "Datasheet" "https://datasheet.lcsc.com/lcsc/1912111437_JILN-JL15EDGK-35002G01_C393013.pdf" (id 3) (at 93.98 133.35 0)
-      (effects (font (size 1.27 1.27)) hide)
-    )
-    (property "LCSC Part Number" "C393013" (id 4) (at 93.98 133.35 0)
+  (symbol (lib_id "Connector:Conn_01x02_Male") (at 133.35 133.35 180) (unit 1)
+    (in_bom yes) (on_board no)
+    (property "Reference" "XSW4" (id 0) (at 128.27 125.73 0))
+    (property "Value" "2pin" (id 1) (at 128.27 128.27 0))
+    (property "Footprint" "" (id 2) (at 133.35 133.35 0)
+      (effects (font (size 1.27 1.27)) hide)
+    )
+    (property "Datasheet" "https://datasheet.lcsc.com/lcsc/1912111437_JILN-JL15EDGK-35002G01_C393013.pdf" (id 3) (at 133.35 133.35 0)
+      (effects (font (size 1.27 1.27)) hide)
+    )
+    (property "LCSC Part Number" "C393013" (id 4) (at 133.35 133.35 0)
       (effects (font (size 1.27 1.27)) hide)
     )
@@
   )
   (symbol (lib_id "Connector:Conn_01x02_Female") (at 133.35 82.55 180) (unit 1)
-    (in_bom yes) (on_board yes) (fields_autoplaced)
-    (property "Reference" "SW2" (id 0) (at 133.985 74.93 0))
-    (property "Value" "2pin" (id 1) (at 133.985 77.47 0))
+    (in_bom yes) (on_board yes)
+    (property "Reference" "SW2" (id 0) (at 135.89 74.93 0))
+    (property "Value" "2pin" (id 1) (at 135.89 77.47 0))
     (property "Footprint" "TerminalBlock_Phoenix:TerminalBlock_Phoenix_PT-1,5-2-3.5-H_1x02_P3.50mm_Horizontal" (id 2) (at 133.35 82.55 0)
       (effects (font (size 1.27 1.27)) hide)
@@
   )
   (symbol (lib_id "Connector:Conn_01x02_Female") (at 133.35 133.35 180) (unit 1)
-    (in_bom yes) (on_board yes) (fields_autoplaced)
-    (property "Reference" "SW4" (id 0) (at 133.985 125.73 0))
-    (property "Value" "2pin" (id 1) (at 133.985 128.27 0))
+    (in_bom yes) (on_board yes)
+    (property "Reference" "SW4" (id 0) (at 135.89 125.73 0))
+    (property "Value" "2pin" (id 1) (at 135.89 128.27 0))
     (property "Footprint" "TerminalBlock_Phoenix:TerminalBlock_Phoenix_PT-1,5-2-3.5-H_1x02_P3.50mm_Horizontal" (id 2) (at 133.35 133.35 0)
       (effects (font (size 1.27 1.27)) hide)

Commit message: ERC, DRC and BOM fixes
Connections:
- no-connect marks 0 -> 8
Changed lines of the file:
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@@
   (junction (at 156.21 101.6) (diameter 0) (color 0 0 0 0)
   )
+  (no_connect (at 128.27 105.41))
+  (no_connect (at 128.27 57.15))
+  (no_connect (at 128.27 80.01))
+  (no_connect (at 128.27 107.95))
+  (no_connect (at 128.27 133.35))
+  (no_connect (at 128.27 130.81))
+  (no_connect (at 128.27 82.55))
+  (no_connect (at 128.27 54.61))
   (wire (pts (xy 149.86 60.96) (xy 156.21 60.96))
     (stroke (width 0) (type default) (color 0 0 0 0))

Commit message: adding project info to sheet frames
Other:
- company: (none) -> makerspace.lt
- title: (none) -> MagLock
Changed lines of the file:
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@@
 (kicad_sch (version 20211123) (generator eeschema)
   (paper "A4")
+  (title_block
+    (title "MagLock")
+    (date "2022-07-20")
+    (rev "2.0")
+    (company "makerspace.lt")
+  )
   (junction (at 149.86 76.2) (diameter 0) (color 0 0 0 0)
   )

Commit message: pulling signal lower on button press. fixes #11
Parts:
- R15, R17, R19, R21: value 10k -> 0
Changed lines of the file:
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@@
       (effects (font (size 1.27 1.27)) (justify left))
     )
-    (property "Value" "10k" (id 1) (at 144.78 101.6 90)
+    (property "Value" "0" (id 1) (at 144.78 101.6 90)
       (effects (font (size 1.27 1.27)) (justify left))
     )
@@
       (effects (font (size 1.27 1.27)) (justify left))
     )
-    (property "Value" "10k" (id 1) (at 144.78 127 90)
+    (property "Value" "0" (id 1) (at 144.78 127 90)
       (effects (font (size 1.27 1.27)) (justify left))
     )
@@
       (effects (font (size 1.27 1.27)) (justify left))
     )
-    (property "Value" "10k" (id 1) (at 144.78 50.8 90)
+    (property "Value" "0" (id 1) (at 144.78 50.8 90)
       (effects (font (size 1.27 1.27)) (justify left))
     )
@@
       (effects (font (size 1.27 1.27)) (justify left))
     )
-    (property "Value" "10k" (id 1) (at 144.78 76.2 90)
-      (effects (font (size 1.27 1.27)) (justify left))
-    )
+    (property "Value" "0" (id 1) (at 144.78 76.2 90)
+      (effects (font (size 1.27 1.27)) (justify left))
+    )

Commit message: using 10V zeners instead of 3V3 in all places. fixes #12, fixes #13
Parts:
- D10, D7, D8, D9: value 3V3 -> 10V; LCSC Part Number C118713 -> C118715
Changed lines of the file:
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@@
       (effects (font (size 1.27 1.27)) (justify left))
     )
-    (property "Value" "3V3" (id 1) (at 156.21 135.89 90)
+    (property "Value" "10V" (id 1) (at 156.21 135.89 90)
       (effects (font (size 1.27 1.27)) (justify left))
     )
@@
       (effects (font (size 1.27 1.27)) hide)
     )
-    (property "Datasheet" "https://datasheet.lcsc.com/lcsc/1806121224_ST-Semtech-MM1Z5226B_C118713.pdf" (id 3) (at 156.21 133.35 0)
-      (effects (font (size 1.27 1.27)) hide)
-    )
-    (property "LCSC Part Number" "C118713" (id 4) (at 156.21 133.35 0)
+    (property "Datasheet" "https://datasheet.lcsc.com/lcsc/1806070724_ST-Semtech-MM1Z5240B_C118715.pdf" (id 3) (at 156.21 133.35 0)
+      (effects (font (size 1.27 1.27)) hide)
+    )
+    (property "LCSC Part Number" "C118715" (id 4) (at 156.21 133.35 0)
       (effects (font (size 1.27 1.27)) hide)
     )
@@
       (effects (font (size 1.27 1.27)) (justify left))
     )
-    (property "Value" "3V3" (id 1) (at 156.21 85.09 90)
+    (property "Value" "10V" (id 1) (at 156.21 85.09 90)
       (effects (font (size 1.27 1.27)) (justify left))
     )
@@
       (effects (font (size 1.27 1.27)) hide)
     )
-    (property "Datasheet" "https://datasheet.lcsc.com/lcsc/1806121224_ST-Semtech-MM1Z5226B_C118713.pdf" (id 3) (at 156.21 82.55 0)
-      (effects (font (size 1.27 1.27)) hide)
-    )
-    (property "LCSC Part Number" "C118713" (id 4) (at 156.21 82.55 0)
+    (property "Datasheet" "https://datasheet.lcsc.com/lcsc/1806070724_ST-Semtech-MM1Z5240B_C118715.pdf" (id 3) (at 156.21 82.55 0)
+      (effects (font (size 1.27 1.27)) hide)
+    )
+    (property "LCSC Part Number" "C118715" (id 4) (at 156.21 82.55 0)
       (effects (font (size 1.27 1.27)) hide)
     )
@@
       (effects (font (size 1.27 1.27)) (justify left))
     )
-    (property "Value" "3V3" (id 1) (at 156.21 59.69 90)
+    (property "Value" "10V" (id 1) (at 156.21 59.69 90)
       (effects (font (size 1.27 1.27)) (justify left))
     )
@@
       (effects (font (size 1.27 1.27)) hide)
     )
-    (property "Datasheet" "https://datasheet.lcsc.com/lcsc/1806121224_ST-Semtech-MM1Z5226B_C118713.pdf" (id 3) (at 156.21 57.15 0)
-      (effects (font (size 1.27 1.27)) hide)
-    )
-    (property "LCSC Part Number" "C118713" (id 4) (at 156.21 57.15 0)
+    (property "Datasheet" "https://datasheet.lcsc.com/lcsc/1806070724_ST-Semtech-MM1Z5240B_C118715.pdf" (id 3) (at 156.21 57.15 0)
+      (effects (font (size 1.27 1.27)) hide)
+    )
+    (property "LCSC Part Number" "C118715" (id 4) (at 156.21 57.15 0)
       (effects (font (size 1.27 1.27)) hide)
     )
@@
       (effects (font (size 1.27 1.27)) (justify left))
     )
-    (property "Value" "3V3" (id 1) (at 156.21 110.49 90)
+    (property "Value" "10V" (id 1) (at 156.21 110.49 90)
       (effects (font (size 1.27 1.27)) (justify left))
     )
@@
       (effects (font (size 1.27 1.27)) hide)
     )
-    (property "Datasheet" "https://datasheet.lcsc.com/lcsc/1806121224_ST-Semtech-MM1Z5226B_C118713.pdf" (id 3) (at 156.21 107.95 0)
-      (effects (font (size 1.27 1.27)) hide)
-    )
-    (property "LCSC Part Number" "C118713" (id 4) (at 156.21 107.95 0)
-      (effects (font (size 1.27 1.27)) hide)
-    )
+    (property "Datasheet" "https://datasheet.lcsc.com/lcsc/1806070724_ST-Semtech-MM1Z5240B_C118715.pdf" (id 3) (at 156.21 107.95 0)
+      (effects (font (size 1.27 1.27)) hide)
+    )
+    (property "LCSC Part Number" "C118715" (id 4) (at 156.21 107.95 0)
+      (effects (font (size 1.27 1.27)) hide)
+    )
