File: _debug_usb_uart.kicad_sch (KiCad schematic)
At the start: 15 parts, among them J1 USB_UART, U1 USBLC6-2SC6, U2 3V3 LDO, U3 CH340C

Commit message: ERC, DRC and BOM fixes
Parts:
- R1, R2: value 5k1 -> 4k7
Changed lines of the file:
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@@
+    (effects (font (size 0.8 0.8)) (justify left bottom))
+  )
+  (label "_DBG_USB_5v" (at 266.7 152.4 0)
     (effects (font (size 0.8 0.8)) (justify left bottom))
   )
@@
       (effects (font (size 1.27 1.27)) (justify left))
     )
-    (property "Value" "5k1" (id 1) (at 118.11 88.9 90)
+    (property "Value" "4k7" (id 1) (at 118.11 88.9 90)
       (effects (font (size 1.27 1.27)) (justify left))
     )
@@
       (effects (font (size 1.27 1.27)) (justify left))
     )
-    (property "Value" "5k1" (id 1) (at 118.11 86.36 90)
+    (property "Value" "4k7" (id 1) (at 118.11 86.36 90)
       (effects (font (size 1.27 1.27)) (justify left))
     )
@@
     (pin "2")
   )
+  (symbol (lib_id "power:PWR_FLAG") (at 266.7 152.4 90) (unit 1)
+    (in_bom yes) (on_board yes) (fields_autoplaced)
+    (property "Reference" "#FLG01" (id 0) (at 264.795 152.4 0)
+      (effects (font (size 1.27 1.27)) hide)
+    )
+    (property "Value" "PWR_FLAG" (id 1) (at 261.62 152.4 0)
+      (effects (font (size 1.27 1.27)) hide)
+    )
+    (property "Footprint" "" (id 2) (at 266.7 152.4 0)
+      (effects (font (size 1.27 1.27)) hide)
+    )
+    (property "Datasheet" "~" (id 3) (at 266.7 152.4 0)
+      (effects (font (size 1.27 1.27)) hide)
+    )
+    (pin "1")
+  )
   (symbol (lib_id "power:GND") (at 154.94 81.28 0) (unit 1)

Commit message: bom and documentation fixes
Parts:
- U3: LCSC Part Number C14267 -> C84681
Changed lines of the file:
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@@
       (effects (font (size 1.27 1.27)) hide)
     )
-    (property "LCSC Part Number" "C14267" (id 4) (at 179.07 110.49 0)
+    (property "LCSC Part Number" "C84681" (id 4) (at 179.07 110.49 0)
       (effects (font (size 1.27 1.27)) hide)
     )

Commit message: adding project info to sheet frames
Other:
- company: (none) -> makerspace.lt
- title: (none) -> MagLock
Changed lines of the file:
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@@
 (kicad_sch (version 20211123) (generator eeschema)
   (paper "A4")
+  (title_block
+    (title "MagLock")
+    (date "2022-07-20")
+    (rev "2.0")
+    (company "makerspace.lt")
+  )
   (junction (at 176.53 73.66) (diameter 0) (color 0 0 0 0)
   )
