File: _usb_ports.kicad_sch (KiCad schematic)
At the start: 11 parts, among them J2 USB, U5 USBLC6-2SC6, U6 USBLC6-2SC6

Commit message: most stuff squeezed on board
Parts:
- F1, F2: symbol Device:Polyfuse -> Device:Fuse
- renumbered C9 to C13, C10 to C14, J2 to J6
Changed lines of the file:
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@@
   (symbol (lib_id "power:GND") (at 162.56 134.62 0) (unit 1)
     (in_bom yes) (on_board yes)
-    (property "Reference" "#PWR022" (id 0) (at 162.56 140.97 0)
+    (property "Reference" "#PWR026" (id 0) (at 162.56 140.97 0)
       (effects (font (size 1.27 1.27)) hide)
     )
@@
   (symbol (lib_id "power:GND") (at 111.76 130.81 0) (unit 1)
     (in_bom yes) (on_board yes)
-    (property "Reference" "#PWR019" (id 0) (at 111.76 137.16 0)
+    (property "Reference" "#PWR023" (id 0) (at 111.76 137.16 0)
       (effects (font (size 1.27 1.27)) hide)
     )
@@
   (symbol (lib_id "power:GND") (at 127 66.04 0) (unit 1)
     (in_bom yes) (on_board yes)
-    (property "Reference" "#PWR020" (id 0) (at 127 72.39 0)
+    (property "Reference" "#PWR024" (id 0) (at 127 72.39 0)
       (effects (font (size 1.27 1.27)) hide)
     )
@@
     (pin "6")
   )
-  (symbol (lib_id "Device:Polyfuse") (at 107.95 50.8 90) (unit 1)
+  (symbol (lib_id "Device:Fuse") (at 107.95 50.8 90) (unit 1)
     (in_bom yes) (on_board yes) (fields_autoplaced)
     (property "Reference" "F1" (id 0) (at 107.95 44.45 90))
     (property "Value" "PTC 300mA" (id 1) (at 107.95 46.99 90))
-    (property "Footprint" "Fuse:Fuse_1206_3216Metric_Pad1.42x1.75mm_HandSolder" (id 2) (at 113.03 49.53 0)
-      (effects (font (size 1.27 1.27)) (justify left) hide)
-    )
-    (property "Datasheet" "https://datasheet.lcsc.com/lcsc/2105241640_Jinrui-Electronic-Materials-Co--JK-nSMD030-16V_C2830239.pdf" (id 3) (at 107.95 50.8 0)
+    (property "Footprint" "Fuse:Fuse_1206_3216Metric_Pad1.42x1.75mm_HandSolder" (id 2) (at 107.95 52.578 90)
+      (effects (font (size 1.27 1.27)) hide)
+    )
+    (property "Datasheet" "~" (id 3) (at 107.95 50.8 0)
       (effects (font (size 1.27 1.27)) hide)
     )
@@
   (symbol (lib_id "power:GND") (at 101.6 66.04 0) (unit 1)
     (in_bom yes) (on_board yes)
-    (property "Reference" "#PWR018" (id 0) (at 101.6 72.39 0)
+    (property "Reference" "#PWR022" (id 0) (at 101.6 72.39 0)
       (effects (font (size 1.27 1.27)) hide)
     )
@@
   (symbol (lib_id "power:GND") (at 195.58 97.79 0) (unit 1)
     (in_bom yes) (on_board yes)
-    (property "Reference" "#PWR023" (id 0) (at 195.58 104.14 0)
+    (property "Reference" "#PWR027" (id 0) (at 195.58 104.14 0)
       (effects (font (size 1.27 1.27)) hide)
     )
@@
   (symbol (lib_id "Device:C") (at 187.96 134.62 90) (unit 1)
     (in_bom yes) (on_board yes)
-    (property "Reference" "C10" (id 0) (at 193.04 133.35 90)
+    (property "Reference" "C14" (id 0) (at 193.04 133.35 90)
       (effects (font (size 1.27 1.27)) (justify left))
     )
@@
     (pin "2")
   )
-  (symbol (lib_id "Device:Polyfuse") (at 133.35 50.8 90) (unit 1)
+  (symbol (lib_id "Device:Fuse") (at 133.35 50.8 90) (unit 1)
     (in_bom yes) (on_board yes) (fields_autoplaced)
     (property "Reference" "F2" (id 0) (at 133.35 44.45 90))
     (property "Value" "PTC 300mA" (id 1) (at 133.35 46.99 90))
-    (property "Footprint" "Fuse:Fuse_1206_3216Metric_Pad1.42x1.75mm_HandSolder" (id 2) (at 138.43 49.53 0)
-      (effects (font (size 1.27 1.27)) (justify left) hide)
-    )
-    (property "Datasheet" "https://datasheet.lcsc.com/lcsc/2105241640_Jinrui-Electronic-Materials-Co--JK-nSMD030-16V_C2830239.pdf" (id 3) (at 133.35 50.8 0)
+    (property "Footprint" "Fuse:Fuse_1206_3216Metric_Pad1.42x1.75mm_HandSolder" (id 2) (at 133.35 52.578 90)
+      (effects (font (size 1.27 1.27)) hide)
+    )
+    (property "Datasheet" "~" (id 3) (at 133.35 50.8 0)
       (effects (font (size 1.27 1.27)) hide)
     )
@@
   (symbol (lib_id "power:GND") (at 195.58 135.89 0) (unit 1)
     (in_bom yes) (on_board yes)
-    (property "Reference" "#PWR024" (id 0) (at 195.58 142.24 0)
+    (property "Reference" "#PWR028" (id 0) (at 195.58 142.24 0)
       (effects (font (size 1.27 1.27)) hide)
     )
@@
   (symbol (lib_id "Connector:USB_A_Stacked") (at 109.22 114.3 0) (unit 1)
     (in_bom yes) (on_board yes) (fields_autoplaced)
-    (property "Reference" "J2" (id 0) (at 109.22 96.52 0))
+    (property "Reference" "J6" (id 0) (at 109.22 96.52 0))
     (property "Value" "USB" (id 1) (at 109.22 99.06 0))
     (property "Footprint" "Connector_USB:USB_A_Wuerth_61400826021_Horizontal_Stacked" (id 2) (at 113.03 128.27 0)
@@
   (symbol (lib_id "Device:C") (at 187.96 96.52 90) (unit 1)
     (in_bom yes) (on_board yes)
-    (property "Reference" "C9" (id 0) (at 193.04 95.25 90)
+    (property "Reference" "C13" (id 0) (at 193.04 95.25 90)
       (effects (font (size 1.27 1.27)) (justify left))
     )
@@
   (symbol (lib_id "power:GND") (at 162.56 96.52 0) (unit 1)
     (in_bom yes) (on_board yes)
-    (property "Reference" "#PWR021" (id 0) (at 162.56 102.87 0)
-      (effects (font (size 1.27 1.27)) hide)
-    )
+    (property "Reference" "#PWR025" (id 0) (at 162.56 102.87 0)
+      (effects (font (size 1.27 1.27)) hide)
+    )

Commit message: general routing finished
Parts:
- renumbered R29 to R31, R30 to R32
Changed lines of the file:
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@@
   (symbol (lib_id "Device:R") (at 127 62.23 0) (unit 1)
     (in_bom yes) (on_board yes)
-    (property "Reference" "R30" (id 0) (at 128.27 60.96 0)
+    (property "Reference" "R32" (id 0) (at 128.27 60.96 0)
       (effects (font (size 1.27 1.27)) (justify left))
     )
@@
   (symbol (lib_id "power:GND") (at 162.56 134.62 0) (unit 1)
     (in_bom yes) (on_board yes)
-    (property "Reference" "#PWR026" (id 0) (at 162.56 140.97 0)
+    (property "Reference" "#PWR027" (id 0) (at 162.56 140.97 0)
       (effects (font (size 1.27 1.27)) hide)
     )
@@
   (symbol (lib_id "power:GND") (at 111.76 130.81 0) (unit 1)
     (in_bom yes) (on_board yes)
-    (property "Reference" "#PWR023" (id 0) (at 111.76 137.16 0)
+    (property "Reference" "#PWR024" (id 0) (at 111.76 137.16 0)
       (effects (font (size 1.27 1.27)) hide)
     )
@@
   (symbol (lib_id "power:GND") (at 127 66.04 0) (unit 1)
     (in_bom yes) (on_board yes)
-    (property "Reference" "#PWR024" (id 0) (at 127 72.39 0)
+    (property "Reference" "#PWR025" (id 0) (at 127 72.39 0)
       (effects (font (size 1.27 1.27)) hide)
     )
@@
   (symbol (lib_id "Device:R") (at 101.6 62.23 0) (unit 1)
     (in_bom yes) (on_board yes)
-    (property "Reference" "R29" (id 0) (at 102.87 60.96 0)
+    (property "Reference" "R31" (id 0) (at 102.87 60.96 0)
       (effects (font (size 1.27 1.27)) (justify left))
     )
@@
   (symbol (lib_id "power:GND") (at 101.6 66.04 0) (unit 1)
     (in_bom yes) (on_board yes)
-    (property "Reference" "#PWR022" (id 0) (at 101.6 72.39 0)
+    (property "Reference" "#PWR023" (id 0) (at 101.6 72.39 0)
       (effects (font (size 1.27 1.27)) hide)
     )
@@
   (symbol (lib_id "power:GND") (at 195.58 97.79 0) (unit 1)
     (in_bom yes) (on_board yes)
-    (property "Reference" "#PWR027" (id 0) (at 195.58 104.14 0)
+    (property "Reference" "#PWR028" (id 0) (at 195.58 104.14 0)
       (effects (font (size 1.27 1.27)) hide)
     )
@@
   (symbol (lib_id "power:GND") (at 195.58 135.89 0) (unit 1)
     (in_bom yes) (on_board yes)
-    (property "Reference" "#PWR028" (id 0) (at 195.58 142.24 0)
+    (property "Reference" "#PWR029" (id 0) (at 195.58 142.24 0)
       (effects (font (size 1.27 1.27)) hide)
     )
@@
   (symbol (lib_id "power:GND") (at 162.56 96.52 0) (unit 1)
     (in_bom yes) (on_board yes)
-    (property "Reference" "#PWR025" (id 0) (at 162.56 102.87 0)
-      (effects (font (size 1.27 1.27)) hide)
-    )
+    (property "Reference" "#PWR026" (id 0) (at 162.56 102.87 0)
+      (effects (font (size 1.27 1.27)) hide)
+    )

Commit message: adding usb port 3d model
Parts:
- J6: footprint Connector_USB:USB_A_Wuerth_61400826021_Horizontal_Stacked -> -local:USB_A_Wuerth_61400826021_Horizontal_Stacked; LCSC Part Number (none) -> C720548
Changed lines of the file:
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@@
     (property "Reference" "J6" (id 0) (at 109.22 96.52 0))
     (property "Value" "USB" (id 1) (at 109.22 99.06 0))
-    (property "Footprint" "Connector_USB:USB_A_Wuerth_61400826021_Horizontal_Stacked" (id 2) (at 113.03 128.27 0)
+    (property "Footprint" "-local:USB_A_Wuerth_61400826021_Horizontal_Stacked" (id 2) (at 113.03 128.27 0)
       (effects (font (size 1.27 1.27)) (justify left) hide)
     )
-    (property "Datasheet" "~" (id 3) (at 114.3 113.03 0)
+    (property "Datasheet" "https://datasheet.lcsc.com/lcsc/2008122034_XUNPU-USB-269-BRW_C720548.pdf" (id 3) (at 114.3 113.03 0)
       (effects (font (size 1.27 1.27)) hide)
     )
-    (property "LCSC Part Number" "~" (id 4) (at 109.22 114.3 0)
+    (property "LCSC Part Number" "C720548" (id 4) (at 109.22 114.3 0)
       (effects (font (size 1.27 1.27)) hide)
     )

Commit message: ERC, DRC and BOM fixes
Changed lines of the file:
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@@
+    (effects (font (size 1.27 1.27)) (justify left bottom))
+  )
+  (label "_VBUS1" (at 165.1 177.8 0)
     (effects (font (size 1.27 1.27)) (justify left bottom))
   )
   (label "_D1+" (at 165.1 144.78 180)
     (effects (font (size 1.27 1.27)) (justify right bottom))
+  )
+  (label "_VBUS2" (at 165.1 180.34 0)
+    (effects (font (size 1.27 1.27)) (justify left bottom))
   )
   (label "_D2+" (at 165.1 124.46 180)
@@
     (pin "1")
   )
+  (symbol (lib_id "power:PWR_FLAG") (at 165.1 180.34 90) (unit 1)
+    (in_bom yes) (on_board yes) (fields_autoplaced)
+    (property "Reference" "#FLG010" (id 0) (at 163.195 180.34 0)
+      (effects (font (size 1.27 1.27)) hide)
+    )
+    (property "Value" "PWR_FLAG" (id 1) (at 160.02 180.34 0)
+      (effects (font (size 1.27 1.27)) hide)
+    )
+    (property "Footprint" "" (id 2) (at 165.1 180.34 0)
+      (effects (font (size 1.27 1.27)) hide)
+    )
+    (property "Datasheet" "~" (id 3) (at 165.1 180.34 0)
+      (effects (font (size 1.27 1.27)) hide)
+    )
+    (pin "1")
+  )
   (symbol (lib_id "power:GND") (at 195.58 97.79 0) (unit 1)
     (in_bom yes) (on_board yes)
@@
     (pin "2")
   )
+  (symbol (lib_id "power:PWR_FLAG") (at 165.1 177.8 90) (unit 1)
+    (in_bom yes) (on_board yes) (fields_autoplaced)
+    (property "Reference" "#FLG09" (id 0) (at 163.195 177.8 0)
+      (effects (font (size 1.27 1.27)) hide)
+    )
+    (property "Value" "PWR_FLAG" (id 1) (at 160.02 177.8 0)
+      (effects (font (size 1.27 1.27)) hide)
+    )
+    (property "Footprint" "" (id 2) (at 165.1 177.8 0)
+      (effects (font (size 1.27 1.27)) hide)
+    )
+    (property "Datasheet" "~" (id 3) (at 165.1 177.8 0)
+      (effects (font (size 1.27 1.27)) hide)
+    )
+    (pin "1")
+  )
   (symbol (lib_id "power:GND") (at 195.58 135.89 0) (unit 1)

Commit message: adding project info to sheet frames
Other:
- company: (none) -> makerspace.lt
- title: (none) -> MagLock
Changed lines of the file:
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@@
 (kicad_sch (version 20211123) (generator eeschema)
   (paper "A4")
+  (title_block
+    (title "MagLock")
+    (date "2022-07-20")
+    (rev "2.0")
+    (company "makerspace.lt")
+  )
   (junction (at 109.22 130.81) (diameter 0) (color 0 0 0 0)
   )

Commit message: reducing PSU and USB power LEDs brightness. fixes #5
Parts:
- R31, R32: value 330 -> 4k7
Changed lines of the file:
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@@
       (effects (font (size 1.27 1.27)) (justify left))
     )
-    (property "Value" "330" (id 1) (at 127 63.5 90)
+    (property "Value" "4k7" (id 1) (at 127 63.5 90)
       (effects (font (size 1.27 1.27)) (justify left))
     )
@@
       (effects (font (size 1.27 1.27)) (justify left))
     )
-    (property "Value" "330" (id 1) (at 101.6 63.5 90)
+    (property "Value" "4k7" (id 1) (at 101.6 63.5 90)
       (effects (font (size 1.27 1.27)) (justify left))
     )
